Commit message: update panther_description | formatting

File: panther_description/urdf/wheel.urdf.xacro (robot description, xacro)
@@ -32,7 +32,7 @@
     </joint>
     <link name="${prefix}_wheel_link">
-       <visual>
+      <visual>
         <geometry>
-            <mesh filename="file://$(find ${wheel_config['mesh_package']})/${wheel_config['folder_path']}/${prefix}_wheel.dae" />
+          <mesh filename="file://$(find ${wheel_config['mesh_package']})/${wheel_config['folder_path']}/${prefix}_wheel.dae" />
         </geometry>
         <origin xyz="0.0 0.0 0.0" rpy="0.0 0.0 0.0" />
@@ -40,10 +40,10 @@
       <collision>
         <geometry>
-            <mesh filename="file://$(find ${wheel_config['mesh_package']})/${wheel_config['folder_path']}/collision.stl" />
+          <mesh filename="file://$(find ${wheel_config['mesh_package']})/${wheel_config['folder_path']}/collision.stl" />
         </geometry>
         <origin xyz="0.0 0.0 0.0" rpy="0.0 0.0 0.0" />
       </collision>
       <inertial>
-        <origin xyz="0.0 ${inertia_y_offset} 0.0" rpy="0.0 0.0 0.0"/>
+        <origin xyz="0.0 ${inertia_y_offset} 0.0" rpy="0.0 0.0 0.0" />
         <mass value="${wheel_config['mass']}" />
         <inertia ixx="${wheel_config['inertia']['ixx']}"
@@ -68,4 +68,11 @@
       <provideFeedback>true</provideFeedback>
     </gazebo>
+    <gazebo reference="${prefix}_wheel_link">
+      <mu1 value="0.8" />
+      <mu2 value="0.8" />
+      <kp value="100000000.0" />
+      <kd value="10.0" />
+      <fdir1 value="1.0 0.0 0.0" />
+    </gazebo>
   </xacro:macro>
 </robot>

Commit message: Fix collisions

File: panther_description/urdf/wheel.urdf.xacro (robot description, xacro)
@@ -44,8 +44,9 @@
       </visual>
       <collision>
-        <origin xyz="0.0 0.0 0.0" rpy="0.0 0.0 0.0" />
+        <origin xyz="0.0 0.0 0.0" rpy="-${pi/2} 0.0 0.0" />
         <geometry>
-          <mesh
-            filename="package://${wheel_config['mesh_package']}/${wheel_config['folder_path']}/wheel_collision.stl" />
+          <cylinder radius="${wheel_config['wheel_radius']}" length="${wheel_config['wheel_width']}"/>
+          <!-- Simulation do not work well with mesh as collision layer. Kept just in case. -->
+          <!-- <mesh filename="package://${wheel_config['mesh_package']}/${wheel_config['folder_path']}/wheel_collision.stl" />  -->
         </geometry>
       </collision>

Commit message: Clean up suggestions

File: panther_description/urdf/wheel.urdf.xacro (robot description, xacro)
@@ -47,6 +47,4 @@
         <geometry>
           <cylinder radius="${wheel_config['wheel_radius']}" length="${wheel_config['wheel_width']}"/>
-          <!-- Simulation do not work well with mesh as collision layer. Kept just in case. -->
-          <!-- <mesh filename="package://${wheel_config['mesh_package']}/${wheel_config['folder_path']}/wheel_collision.stl" />  -->
         </geometry>
       </collision>

Commit message: Added mecanum argument | added y friction to normal wheels
Signed-off-by: Jakub Delicat <jakub.delicat@husarion.com>

File: panther_description/urdf/wheel.urdf.xacro (robot description, xacro)
@@ -62,17 +62,19 @@
     </link>
     <xacro:if value="${use_sim}">
-      <gazebo reference="${prefix}_wheel_link" xmlns:ignition="http://ignitionrobotics.org/schema">
-        <collision>
-          <surface>
-            <friction>
-              <ode>
-                <mu>1.0</mu>
-                <mu2>0.0</mu2>
-                <fdir1 ignition:expressed_in="base_link">${fdir}</fdir1>
-              </ode>
-            </friction>
-          </surface>
-        </collision>
-      </gazebo>
+      <xacro:if value="${wheel_config['mecanum']}">
+        <gazebo reference="${prefix}_wheel_link" xmlns:ignition="http://ignitionrobotics.org/schema">
+          <collision>
+            <surface>
+              <friction>
+                <ode>
+                  <mu>1.0</mu>
+                  <mu2>0.0</mu2>
+                  <fdir1 ignition:expressed_in="base_link">${fdir}</fdir1>
+                </ode>
+              </friction>
+            </surface>
+          </collision>
+        </gazebo>
+      </xacro:if>
     </xacro:if>
   </xacro:macro>
