Commit message: add ros-control (#50)
* add ros-control

* fix indents

* Update panther_gazebo/config/panther_ros_controler.yaml

Co-authored-by: Dawid Kmak <73443304+KmakD@users.noreply.github.com>

* Update panther_gazebo/config/panther_ros_controler.yaml

Co-authored-by: Dawid Kmak <73443304+KmakD@users.noreply.github.com>

* Update panther_gazebo/config/panther_ros_controler.yaml

Co-authored-by: Dawid Kmak <73443304+KmakD@users.noreply.github.com>

* Update panther_gazebo/launch/panther_spawn.launch

Co-authored-by: Dawid Kmak <73443304+KmakD@users.noreply.github.com>

* Update panther_gazebo/launch/panther_spawn.launch

Co-authored-by: Dawid Kmak <73443304+KmakD@users.noreply.github.com>

* Update panther_spawn.launch

* Update panther_spawn.launch

* Update panther_spawn.launch

* Update panther_spawn.launch

---------

Co-authored-by: Dawid Kmak <73443304+KmakD@users.noreply.github.com>

File: panther_description/urdf/panther_macro.urdf.xacro (robot description, xacro)
@@ -11,10 +11,17 @@
                        imu_rot_y:=0.0
                        wheel_config_path:=None
-                       simulation_engine:='gazebo-classic'">
+                       simulation_engine:='gazebo-classic'
+                       use_ros_control:=false">
     <xacro:if value="${wheel_config_path == 'None'}">
-      <xacro:property name="wheel_config_file" value="$(find panther_description)/config/WH01.yaml"  />
+      <xacro:property name="wheel_config_file" value="$(find panther_description)/config/WH01.yaml" />
     </xacro:if>
     <xacro:unless value="${wheel_config_path == 'None'}">
-      <xacro:property name="wheel_config_file" value="$(arg wheel_config_path)"  />
+      <xacro:property name="wheel_config_file" value="$(arg wheel_config_path)" />
+    </xacro:unless>
+    <xacro:if value="${use_ros_control}">
+      <xacro:property name="hardware_interface" value="VelocityJointInterface" />
+    </xacro:if>
+    <xacro:unless value="${use_ros_control}">
+      <xacro:property name="hardware_interface" value="EffortJointInterface" />
     </xacro:unless>
     <xacro:property name="wheel_config" value="${xacro.load_yaml(wheel_config_file)}" />
@@ -37,60 +44,64 @@
       wheel_config="${wheel_config}"
       wheel_separation_x="${wheel_separation_x}"
+      hardware_interface="${hardware_interface}"
       prefix="fl" />
     <xacro:wheel.wheel
       wheel_config="${wheel_config}"
       wheel_separation_x="${wheel_separation_x}"
+      hardware_interface="${hardware_interface}"
       prefix="fr" />
     <xacro:wheel.wheel
       wheel_config="${wheel_config}"
       wheel_separation_x="${wheel_separation_x}"
+      hardware_interface="${hardware_interface}"
       prefix="rl" />
     <xacro:wheel.wheel
       wheel_config="${wheel_config}"
       wheel_separation_x="${wheel_separation_x}"
+      hardware_interface="${hardware_interface}"
       prefix="rr" />
     <xacro:if value="${simulation_engine == 'gazebo-classic'}">
       <gazebo>
         <plugin name="gazebo_ros_control" filename="libgazebo_ros_control.so">
-          <robotNamespace>/</robotNamespace>
-          <legacyModeNS>true</legacyModeNS>
         </plugin>
       </gazebo>
-      <xacro:if value="${wheel_config['kinematics'] == 'differential'}">
-        <gazebo>
-          <plugin name='skid_steer_drive_controller' filename='libgazebo_ros_skid_steer_drive.so'>
-            <updateRate>20.0</updateRate>
-            <robotBaseFrame>base_link</robotBaseFrame>
-            <wheelSeparation>${wheel_config['wheel_separation']}</wheelSeparation>
-            <wheelDiameter>${wheel_config['wheel_radius']*2.0}</wheelDiameter>
-            <torque>34.5</torque>
-            <leftFrontJoint>fl_wheel_joint</leftFrontJoint>
-            <rightFrontJoint>fr_wheel_joint</rightFrontJoint>
-            <leftRearJoint>rl_wheel_joint</leftRearJoint>
-            <rightRearJoint>rr_wheel_joint</rightRearJoint>
-            <topicName>cmd_vel</topicName>
-            <commandTopic>cmd_vel</commandTopic>
-            <broadcastTF>true</broadcastTF>
-            <odometryTopic>odom</odometryTopic>
-            <odometryFrame>odom</odometryFrame>
-            <covariance_x>0.0001</covariance_x>
-            <covariance_y>0.0001</covariance_y>
-            <covariance_yaw>0.0100</covariance_yaw>
-          </plugin>
-        </gazebo>
-      </xacro:if>
-      <xacro:if value="${wheel_config['kinematics'] == 'mecanum'}">
-        <gazebo>
-          <plugin name="object_controller" filename="libgazebo_ros_planar_move.so">
-            <commandTopic>cmd_vel</commandTopic>
-            <odometryTopic>odom</odometryTopic>
-            <odometryFrame>odom</odometryFrame>
-            <odometryRate>20.0</odometryRate>
-            <robotBaseFrame>base_link</robotBaseFrame>
-            <cmdTimeout>-1</cmdTimeout>
-          </plugin>
-        </gazebo>
-      </xacro:if>
-  </xacro:if>
+      <xacro:unless value="${use_ros_control}">
+        <xacro:if value="${wheel_config['kinematics'] == 'differential'}">
+          <gazebo>
+            <plugin name='skid_steer_drive_controller' filename='libgazebo_ros_skid_steer_drive.so'>
+              <updateRate>20.0</updateRate>
+              <robotBaseFrame>base_link</robotBaseFrame>
+              <wheelSeparation>${wheel_config['wheel_separation']}</wheelSeparation>
+              <wheelDiameter>${wheel_config['wheel_radius']*2.0}</wheelDiameter>
+              <torque>34.5</torque>
+              <leftFrontJoint>fl_wheel_joint</leftFrontJoint>
+              <rightFrontJoint>fr_wheel_joint</rightFrontJoint>
+              <leftRearJoint>rl_wheel_joint</leftRearJoint>
+              <rightRearJoint>rr_wheel_joint</rightRearJoint>
+              <topicName>cmd_vel</topicName>
+              <commandTopic>cmd_vel</commandTopic>
+              <broadcastTF>true</broadcastTF>
+              <odometryTopic>odom</odometryTopic>
+              <odometryFrame>odom</odometryFrame>
+              <covariance_x>0.0001</covariance_x>
+              <covariance_y>0.0001</covariance_y>
+              <covariance_yaw>0.0100</covariance_yaw>
+            </plugin>
+          </gazebo>
+        </xacro:if>
+        <xacro:if value="${wheel_config['kinematics'] == 'mecanum'}">
+          <gazebo>
+            <plugin name="object_controller" filename="libgazebo_ros_planar_move.so">
+              <commandTopic>cmd_vel</commandTopic>
+              <odometryTopic>odom</odometryTopic>
+              <odometryFrame>odom</odometryFrame>
+              <odometryRate>20.0</odometryRate>
+              <robotBaseFrame>base_link</robotBaseFrame>
+              <cmdTimeout>-1</cmdTimeout>
+            </plugin>
+          </gazebo>
+        </xacro:if>
+      </xacro:unless>
+    </xacro:if>
   </xacro:macro>
 </robot>

Commit message: Added exporting interfaces test
Signed-off-by: Jakub Delicat <jakub.delicat@husarion.com>

File: panther_description/urdf/panther_macro.urdf.xacro (robot description, xacro)
@@ -58,81 +58,4 @@
       wheel_separation_x="${wheel_separation_x}"
       prefix="rr" />
-    <ros2_control name="wheels" type="system">
-      <hardware>
-        <xacro:if value="${use_sim}">
-          <xacro:if value="${simulation_engine == 'ignition-gazebo'}">
-            <plugin>ign_ros2_control/IgnitionSystem</plugin>
-          </xacro:if>
-        </xacro:if>
-        <xacro:unless value="$(arg use_sim)">
-          <plugin>panther_hardware_interfaces/PantherSystem</plugin>
-          <param name="panther_version">${panther_version}</param>
-          <param name="encoder_resolution">1600</param>
-          <param name="gear_ratio">30.08</param>
-          <param name="gearbox_efficiency">0.75</param>
-          <!-- Same as set in the Roboteq driver (TNM parameter) -->
-          <param name="motor_torque_constant">0.11</param>
-          <!-- Max RPM speed set in the Roboteq driver (MXRPM parameter) -->
-          <param name="max_rpm_motor_speed">3600.0</param>
-          <param name="can_interface_name">panther_can</param>
-          <param name="master_can_id">3</param>
-          <param name="front_driver_can_id">1</param>
-          <param name="rear_driver_can_id">2</param>
-          <param name="sdo_operation_timeout_ms">100</param>
-          <!-- Depends on frequency of the controller, more critical motors state are sent with
-           higher frequency, other parameters are sent with lower, here allowed time is set
-           to be expected period +50% margin -->
-          <param name="pdo_motor_states_timeout_ms">15</param>
-          <param name="pdo_driver_state_timeout_ms">75</param>
-          <!-- It will be rounded to the closest value taking into account current controller frequency -->
-          <param name="driver_states_update_frequency">20.0</param>
-          <param name="max_roboteq_initialization_attempts">5</param>
-          <param name="max_roboteq_activation_attempts">5</param>
-          <param name="max_safety_stop_attempts">20</param>
-          <!-- TODO after all tests update parameters, these ones are quite high for the worst case scenario -->
-          <param name="max_write_pdo_cmds_errors_count">4</param>
-          <param name="max_read_pdo_motor_states_errors_count">4</param>
-          <param name="max_read_pdo_driver_state_errors_count">20</param>
-        </xacro:unless>
-      </hardware>
-      <joint name="fl_wheel_joint">
-        <command_interface name="velocity" />
-        <state_interface name="position" />
-        <state_interface name="velocity" />
-        <state_interface name="effort" />
-      </joint>
-      <joint name="fr_wheel_joint">
-        <command_interface name="velocity" />
-        <state_interface name="position" />
-        <state_interface name="velocity" />
-        <state_interface name="effort" />
-      </joint>
-      <joint name="rl_wheel_joint">
-        <command_interface name="velocity" />
-        <state_interface name="position" />
-        <state_interface name="velocity" />
-        <state_interface name="effort" />
-      </joint>
-      <joint name="rr_wheel_joint">
-        <command_interface name="velocity" />
-        <state_interface name="position" />
-        <state_interface name="velocity" />
-        <state_interface name="effort" />
-      </joint>
-      <xacro:if value="${use_sim}">
-        <sensor name="imu">
-          <state_interface name="orientation.x" />
-          <state_interface name="orientation.y" />
-          <state_interface name="orientation.z" />
-          <state_interface name="orientation.w" />
-          <state_interface name="angular_velocity.x" />
-          <state_interface name="angular_velocity.y" />
-          <state_interface name="angular_velocity.z" />
-          <state_interface name="linear_acceleration.x" />
-          <state_interface name="linear_acceleration.y" />
-          <state_interface name="linear_acceleration.z" />
-        </sensor>
-      </xacro:if>
-    </ros2_control>
     <xacro:unless value="$(arg use_sim)">
       <ros2_control name="imu" type="sensor">

Commit message: Add IMU noise

File: panther_description/urdf/panther_macro.urdf.xacro (robot description, xacro)
@@ -16,19 +16,8 @@
             simulation_engine:='ignition-gazebo'">
     <xacro:property name="wheel_config" value="${xacro.load_yaml(wheel_config_file)}" />
-    <xacro:if value="${use_sim}">
-      <xacro:property name="battery_config" value="${xacro.load_yaml(battery_config_file)}" />
-      <xacro:property name="bat_initial_charge"
-        value="${20.0*battery_config['initial_charge_percentage']/100.0}" />
-      <xacro:property name="bat_charging_time" value="${battery_config['charging_time']}" />
-      <xacro:if value="${battery_config['simulate_discharging']}">
-        <xacro:property name="bat_power_load" value="${battery_config['power_load']}" />
-      </xacro:if>
-      <xacro:unless value="${battery_config['simulate_discharging']}">
-        <xacro:property name="bat_power_load" value="0.0" />
-      </xacro:unless>
-    </xacro:if>
     <xacro:property name="wheel_separation_x" value="0.44" />
     <!-- INCLUDE ROBOT PARTS DEFINITIONS -->
     <xacro:include filename="$(find panther_description)/urdf/body.urdf.xacro" ns="body" />
+    <xacro:include filename="$(find panther_description)/urdf/gazebo.urdf.xacro" ns="gazebo" />
     <xacro:include filename="$(find panther_description)/urdf/wheel.urdf.xacro" ns="wheel" />
     <!-- BODY DECLARATION -->
@@ -120,45 +109,7 @@
     </ros2_control>
     <xacro:if value="${use_sim}">
-      <gazebo>
-        <plugin filename="ign_ros2_control-system"
-          name="ign_ros2_control::IgnitionROS2ControlPlugin">
-          <parameters>${controller_config_file}</parameters>
-          <ros>
-            <remapping>/panther_base_controller/cmd_vel_unstamped:=/cmd_vel</remapping>
-          </ros>
-        </plugin>
-      </gazebo>
-      <gazebo>
-        <plugin filename="ignition-gazebo-linearbatteryplugin-system"
-          name="gz::sim::systems::LinearBatteryPlugin">
-          <battery_name>panther_battery</battery_name>
-          <voltage>41.4</voltage>
-          <open_circuit_voltage_constant_coef>42.0</open_circuit_voltage_constant_coef>
-          <open_circuit_voltage_linear_coef>-10.0</open_circuit_voltage_linear_coef>
-          <initial_charge>${bat_initial_charge}</initial_charge>
-          <capacity>20.0</capacity>
-          <resistance>0.15</resistance>
-          <smooth_current_tau>2.0</smooth_current_tau>
-          <enable_recharge>true</enable_recharge>
-          <charging_time>${bat_charging_time}</charging_time>
-          <soc_threshold>2.0</soc_threshold>
-          <power_load>${bat_power_load}</power_load>
-          <start_on_motion>false</start_on_motion>
-          <!-- https://github.com/gazebosim/gz-sim/issues/225 -->
-          <fix_issue_225>true</fix_issue_225>
-        </plugin>
-      </gazebo>
-      <gazebo reference="imu_link">
-        <sensor name="imu" type="imu">
-          <plugin filename="ignition-gazebo-imu-system" name="ignition::gazebo::systems::Imu" />
-          <always_on>true</always_on>
-          <update_rate>100</update_rate>
-          <topic>imu/data_raw</topic>
-          <visualize>false</visualize>
-          <enable_metrics>false</enable_metrics>
-          <frame_id>imu_link</frame_id>
-          <ignition_frame_id>imu_link</ignition_frame_id>
-        </sensor>
-      </gazebo>
+      <xacro:gazebo.battery config_file="${battery_config_file}"/>
+      <xacro:gazebo.controller config_file="${controller_config_file}"/>
+      <xacro:gazebo.imu reference_frame="imu_link" name="imu"/>
     </xacro:if>
   </xacro:macro>

Commit message: Add IMU noise + basic EKF configuration (#229)
* Fix collisions

* remove parent dir

* Add IMU noise

* EKF working

* Add controller

* Update panther_bringup/config/ekf.yaml

* Update panther_bringup/config/ekf.yaml

* Format

File: panther_description/urdf/panther_macro.urdf.xacro (robot description, xacro)
@@ -16,19 +16,8 @@
             simulation_engine:='ignition-gazebo'">
     <xacro:property name="wheel_config" value="${xacro.load_yaml(wheel_config_file)}" />
-    <xacro:if value="${use_sim}">
-      <xacro:property name="battery_config" value="${xacro.load_yaml(battery_config_file)}" />
-      <xacro:property name="bat_initial_charge"
-        value="${20.0*battery_config['initial_charge_percentage']/100.0}" />
-      <xacro:property name="bat_charging_time" value="${battery_config['charging_time']}" />
-      <xacro:if value="${battery_config['simulate_discharging']}">
-        <xacro:property name="bat_power_load" value="${battery_config['power_load']}" />
-      </xacro:if>
-      <xacro:unless value="${battery_config['simulate_discharging']}">
-        <xacro:property name="bat_power_load" value="0.0" />
-      </xacro:unless>
-    </xacro:if>
     <xacro:property name="wheel_separation_x" value="0.44" />
     <!-- INCLUDE ROBOT PARTS DEFINITIONS -->
     <xacro:include filename="$(find panther_description)/urdf/body.urdf.xacro" ns="body" />
+    <xacro:include filename="$(find panther_description)/urdf/gazebo.urdf.xacro" ns="gazebo" />
     <xacro:include filename="$(find panther_description)/urdf/wheel.urdf.xacro" ns="wheel" />
     <!-- BODY DECLARATION -->
@@ -120,45 +109,7 @@
     </ros2_control>
     <xacro:if value="${use_sim}">
-      <gazebo>
-        <plugin filename="ign_ros2_control-system"
-          name="ign_ros2_control::IgnitionROS2ControlPlugin">
-          <parameters>${controller_config_file}</parameters>
-          <ros>
-            <remapping>/panther_base_controller/cmd_vel_unstamped:=/cmd_vel</remapping>
-          </ros>
-        </plugin>
-      </gazebo>
-      <gazebo>
-        <plugin filename="ignition-gazebo-linearbatteryplugin-system"
-          name="gz::sim::systems::LinearBatteryPlugin">
-          <battery_name>panther_battery</battery_name>
-          <voltage>41.4</voltage>
-          <open_circuit_voltage_constant_coef>42.0</open_circuit_voltage_constant_coef>
-          <open_circuit_voltage_linear_coef>-10.0</open_circuit_voltage_linear_coef>
-          <initial_charge>${bat_initial_charge}</initial_charge>
-          <capacity>20.0</capacity>
-          <resistance>0.15</resistance>
-          <smooth_current_tau>2.0</smooth_current_tau>
-          <enable_recharge>true</enable_recharge>
-          <charging_time>${bat_charging_time}</charging_time>
-          <soc_threshold>2.0</soc_threshold>
-          <power_load>${bat_power_load}</power_load>
-          <start_on_motion>false</start_on_motion>
-          <!-- https://github.com/gazebosim/gz-sim/issues/225 -->
-          <fix_issue_225>true</fix_issue_225>
-        </plugin>
-      </gazebo>
-      <gazebo reference="imu_link">
-        <sensor name="imu" type="imu">
-          <plugin filename="ignition-gazebo-imu-system" name="ignition::gazebo::systems::Imu" />
-          <always_on>true</always_on>
-          <update_rate>100</update_rate>
-          <topic>imu/data_raw</topic>
-          <visualize>false</visualize>
-          <enable_metrics>false</enable_metrics>
-          <frame_id>imu_link</frame_id>
-          <ignition_frame_id>imu_link</ignition_frame_id>
-        </sensor>
-      </gazebo>
+      <xacro:gazebo.battery config_file="${battery_config_file}" />
+      <xacro:gazebo.controller config_file="${controller_config_file}" />
+      <xacro:gazebo.imu reference_frame="imu_link" name="imu" />
     </xacro:if>
   </xacro:macro>

Commit message: revert roboteqs
Signed-off-by: Jakub Delicat <jakub.delicat@husarion.com>

File: panther_description/urdf/panther_macro.urdf.xacro (robot description, xacro)
@@ -47,4 +47,80 @@
       wheel_separation_x="${wheel_separation_x}"
       prefix="rr" />
+    <ros2_control name="wheels" type="system">
+      <hardware>
+        <xacro:if value="${use_sim}">
+          <xacro:if value="${simulation_engine == 'ignition-gazebo'}">
+            <plugin>ign_ros2_control/IgnitionSystem</plugin>
+          </xacro:if>
+        </xacro:if>
+        <xacro:unless value="$(arg use_sim)">
+          <plugin>panther_hardware_interfaces/PantherSystem</plugin>
+          <param name="panther_version">${panther_version}</param>
+          <param name="encoder_resolution">1600</param>
+          <param name="gear_ratio">30.08</param>
+          <param name="gearbox_efficiency">0.75</param>
+          <!-- Same as set in the Roboteq driver (TNM parameter) -->
+          <param name="motor_torque_constant">0.11</param>
+          <!-- Max RPM speed set in the Roboteq driver (MXRPM parameter) -->
+          <param name="max_rpm_motor_speed">3600.0</param>
+          <param name="can_interface_name">panther_can</param>
+          <param name="master_can_id">3</param>
+          <param name="front_driver_can_id">1</param>
+          <param name="rear_driver_can_id">2</param>
+          <param name="sdo_operation_timeout_ms">100</param>
+          <!-- Depends on frequency of the controller, more critical motors state are sent with
+           higher frequency, other parameters are sent with lower, here allowed time is set
+           to be expected period +50% margin -->
+          <param name="pdo_motor_states_timeout_ms">15</param>
+          <param name="pdo_driver_state_timeout_ms">75</param>
+          <!-- It will be rounded to the closest value taking into account current controller frequency -->
+          <param name="driver_states_update_frequency">20.0</param>
+          <param name="max_roboteq_initialization_attempts">5</param>
+          <param name="max_roboteq_activation_attempts">5</param>
+          <!-- TODO after all tests update parameters, these ones are quite high for the worst case scenario -->
+          <param name="max_write_pdo_cmds_errors_count">4</param>
+          <param name="max_read_pdo_motor_states_errors_count">4</param>
+          <param name="max_read_pdo_driver_state_errors_count">20</param>
+        </xacro:unless>
+      </hardware>
+      <joint name="fl_wheel_joint">
+        <command_interface name="velocity" />
+        <state_interface name="position" />
+        <state_interface name="velocity" />
+        <state_interface name="effort" />
+      </joint>
+      <joint name="fr_wheel_joint">
+        <command_interface name="velocity" />
+        <state_interface name="position" />
+        <state_interface name="velocity" />
+        <state_interface name="effort" />
+      </joint>
+      <joint name="rl_wheel_joint">
+        <command_interface name="velocity" />
+        <state_interface name="position" />
+        <state_interface name="velocity" />
+        <state_interface name="effort" />
+      </joint>
+      <joint name="rr_wheel_joint">
+        <command_interface name="velocity" />
+        <state_interface name="position" />
+        <state_interface name="velocity" />
+        <state_interface name="effort" />
+      </joint>
+      <xacro:if value="${use_sim}">
+        <sensor name="imu">
+          <state_interface name="orientation.x" />
+          <state_interface name="orientation.y" />
+          <state_interface name="orientation.z" />
+          <state_interface name="orientation.w" />
+          <state_interface name="angular_velocity.x" />
+          <state_interface name="angular_velocity.y" />
+          <state_interface name="angular_velocity.z" />
+          <state_interface name="linear_acceleration.x" />
+          <state_interface name="linear_acceleration.y" />
+          <state_interface name="linear_acceleration.z" />
+        </sensor>
+      </xacro:if>
+    </ros2_control>
     <xacro:unless value="$(arg use_sim)">
       <ros2_control name="imu" type="sensor">
