Commit message: add ros-control

File: panther_description/urdf/panther.urdf.xacro (robot description, xacro)
@@ -12,4 +12,5 @@
   <xacro:arg name="wheel_config_path" default="$(find panther_description)/config/WH01.yaml" />
   <xacro:arg name="simulation_engine" default="gazebo-classic" />
+  <xacro:arg name="use_ros_control" default="false" />
   <xacro:include filename="$(find panther_description)/urdf/panther_macro.urdf.xacro" ns="husarion" />
   <xacro:husarion.panther_robot
@@ -23,4 +24,5 @@
     imu_rot_y="$(arg imu_rot_y)"
     wheel_config_path="$(arg wheel_config_path)"
-    simulation_engine="$(arg simulation_engine)" />
+    simulation_engine="$(arg simulation_engine)"
+    use_ros_control="$(arg use_ros_control)" />
 </robot>

File: panther_description/urdf/panther_macro.urdf.xacro (robot description, xacro)
@@ -2,5 +2,5 @@
 <robot xmlns:xacro="http://wiki.ros.org/xacro">
   <xacro:macro name="panther_robot"
-               params="use_sim:=false
+    params="use_sim:=false
                        dual_bat:=false
                        imu_pos_x:=0.168
@@ -11,10 +11,17 @@
                        imu_rot_y:=0.0
                        wheel_config_path:=None
-                       simulation_engine:='gazebo-classic'">
+                       simulation_engine:='gazebo-classic'
+                       use_ros_control:=false">
     <xacro:if value="${wheel_config_path == 'None'}">
-      <xacro:property name="wheel_config_file" value="$(find panther_description)/config/WH01.yaml"  />
+      <xacro:property name="wheel_config_file" value="$(find panther_description)/config/WH01.yaml" />
     </xacro:if>
     <xacro:unless value="${wheel_config_path == 'None'}">
-      <xacro:property name="wheel_config_file" value="$(arg wheel_config_path)"  />
+      <xacro:property name="wheel_config_file" value="$(arg wheel_config_path)" />
+    </xacro:unless>
+    <xacro:if value="${use_ros_control}">
+      <xacro:property name="hardware_interface" value="VelocityJointInterface" />
+    </xacro:if>
+    <xacro:unless value="${use_ros_control}">
+      <xacro:property name="hardware_interface" value="EffortJointInterface" />
     </xacro:unless>
     <xacro:property name="wheel_config" value="${xacro.load_yaml(wheel_config_file)}" />
@@ -37,60 +44,64 @@
       wheel_config="${wheel_config}"
       wheel_separation_x="${wheel_separation_x}"
+      hardware_interface="${hardware_interface}"
       prefix="fl" />
     <xacro:wheel.wheel
       wheel_config="${wheel_config}"
       wheel_separation_x="${wheel_separation_x}"
+      hardware_interface="${hardware_interface}"
       prefix="fr" />
     <xacro:wheel.wheel
       wheel_config="${wheel_config}"
       wheel_separation_x="${wheel_separation_x}"
+      hardware_interface="${hardware_interface}"
       prefix="rl" />
     <xacro:wheel.wheel
       wheel_config="${wheel_config}"
       wheel_separation_x="${wheel_separation_x}"
+      hardware_interface="${hardware_interface}"
       prefix="rr" />
     <xacro:if value="${simulation_engine == 'gazebo-classic'}">
       <gazebo>
         <plugin name="gazebo_ros_control" filename="libgazebo_ros_control.so">
-          <robotNamespace>/</robotNamespace>
-          <legacyModeNS>true</legacyModeNS>
         </plugin>
       </gazebo>
-      <xacro:if value="${wheel_config['kinematics'] == 'differential'}">
-        <gazebo>
-          <plugin name='skid_steer_drive_controller' filename='libgazebo_ros_skid_steer_drive.so'>
-            <updateRate>20.0</updateRate>
-            <robotBaseFrame>base_link</robotBaseFrame>
-            <wheelSeparation>${wheel_config['wheel_separation']}</wheelSeparation>
-            <wheelDiameter>${wheel_config['wheel_radius']*2.0}</wheelDiameter>
-            <torque>34.5</torque>
-            <leftFrontJoint>fl_wheel_joint</leftFrontJoint>
-            <rightFrontJoint>fr_wheel_joint</rightFrontJoint>
-            <leftRearJoint>rl_wheel_joint</leftRearJoint>
-            <rightRearJoint>rr_wheel_joint</rightRearJoint>
-            <topicName>cmd_vel</topicName>
-            <commandTopic>cmd_vel</commandTopic>
-            <broadcastTF>true</broadcastTF>
-            <odometryTopic>odom</odometryTopic>
-            <odometryFrame>odom</odometryFrame>
-            <covariance_x>0.0001</covariance_x>
-            <covariance_y>0.0001</covariance_y>
-            <covariance_yaw>0.0100</covariance_yaw>
-          </plugin>
-        </gazebo>
-      </xacro:if>
-      <xacro:if value="${wheel_config['kinematics'] == 'mecanum'}">
-        <gazebo>
-          <plugin name="object_controller" filename="libgazebo_ros_planar_move.so">
-            <commandTopic>cmd_vel</commandTopic>
-            <odometryTopic>odom</odometryTopic>
-            <odometryFrame>odom</odometryFrame>
-            <odometryRate>20.0</odometryRate>
-            <robotBaseFrame>base_link</robotBaseFrame>
-            <cmdTimeout>-1</cmdTimeout>
-          </plugin>
-        </gazebo>
-      </xacro:if>
-  </xacro:if>
+      <xacro:unless value="${use_ros_control}">
+        <xacro:if value="${wheel_config['kinematics'] == 'differential'}">
+          <gazebo>
+            <plugin name='skid_steer_drive_controller' filename='libgazebo_ros_skid_steer_drive.so'>
+              <updateRate>20.0</updateRate>
+              <robotBaseFrame>base_link</robotBaseFrame>
+              <wheelSeparation>${wheel_config['wheel_separation']}</wheelSeparation>
+              <wheelDiameter>${wheel_config['wheel_radius']*2.0}</wheelDiameter>
+              <torque>34.5</torque>
+              <leftFrontJoint>fl_wheel_joint</leftFrontJoint>
+              <rightFrontJoint>fr_wheel_joint</rightFrontJoint>
+              <leftRearJoint>rl_wheel_joint</leftRearJoint>
+              <rightRearJoint>rr_wheel_joint</rightRearJoint>
+              <topicName>cmd_vel</topicName>
+              <commandTopic>cmd_vel</commandTopic>
+              <broadcastTF>true</broadcastTF>
+              <odometryTopic>odom</odometryTopic>
+              <odometryFrame>odom</odometryFrame>
+              <covariance_x>0.0001</covariance_x>
+              <covariance_y>0.0001</covariance_y>
+              <covariance_yaw>0.0100</covariance_yaw>
+            </plugin>
+          </gazebo>
+        </xacro:if>
+        <xacro:if value="${wheel_config['kinematics'] == 'mecanum'}">
+          <gazebo>
+            <plugin name="object_controller" filename="libgazebo_ros_planar_move.so">
+              <commandTopic>cmd_vel</commandTopic>
+              <odometryTopic>odom</odometryTopic>
+              <odometryFrame>odom</odometryFrame>
+              <odometryRate>20.0</odometryRate>
+              <robotBaseFrame>base_link</robotBaseFrame>
+              <cmdTimeout>-1</cmdTimeout>
+            </plugin>
+          </gazebo>
+        </xacro:if>
+      </xacro:unless>
+    </xacro:if>
   </xacro:macro>
 </robot>

File: panther_description/urdf/wheel.urdf.xacro (robot description, xacro)
@@ -2,5 +2,5 @@
 <robot xmlns:xacro="http://www.ros.org/wiki/xacro">
   <!-- wheel defining macro -->
-  <xacro:macro name="wheel" params="wheel_config prefix wheel_separation_x">
+  <xacro:macro name="wheel" params="wheel_config wheel_separation_x hardware_interface prefix">
     <xacro:if value="${prefix == 'fl'}">
       <xacro:property name="x" value="${wheel_separation_x/2.0}" />
@@ -58,9 +58,9 @@
       <type>transmission_interface/SimpleTransmission</type>
       <joint name="${prefix}_wheel_joint">
-        <hardwareInterface>hardware_interface/EffortJointInterface</hardwareInterface>
+        <hardwareInterface>hardware_interface/${hardware_interface}</hardwareInterface>
       </joint>
       <actuator name="${prefix}_wheel_actuator">
         <mechanicalReduction>1</mechanicalReduction>
-        <hardwareInterface>hardware_interface/EffortJointInterface</hardwareInterface>
+        <hardwareInterface>hardware_interface/${hardware_interface}</hardwareInterface>
       </actuator>
     </transmission>

Commit message: Reduce merge x y z  together

File: panther_description/urdf/panther.urdf.xacro (robot description, xacro)
@@ -5,4 +5,6 @@
   <!-- if lidars have to work correctly, use_gpu has to be true. -->
   <xacro:arg name="use_gpu" default="true" />
+  <xacro:arg name="imu_xyz" default="0.169 0.025 0.092" />
+  <xacro:arg name="imu_rpy" default="0.0 0.0 -1.57" />
   <xacro:arg name="wheel_config_file"
     default="$(find panther_description)/config/WH01.yaml" />
@@ -16,4 +18,6 @@
     panther_version="$(arg panther_version)"
     use_sim="$(arg use_sim)"
+    imu_xyz="$(arg imu_xyz)"
+    imu_rpy="$(arg imu_rpy)"
     wheel_config_file="$(arg wheel_config_file)"
     controller_config_file="$(arg controller_config_file)"

File: panther_description/urdf/panther_macro.urdf.xacro (robot description, xacro)
@@ -8,10 +8,8 @@
             battery_config_file
             use_sim:=false
+            imu_xyz:='0.169 0.025 0.092'
+            imu_rpy:='0.0 0.0 -1.57'
             namespace:=''">
-    <xacro:if value="${float(panther_version) >= 1.0}" >
-      <xacro:property name="imu_xyz" value="0.168 0.028 0.083" lazy_eval="false"/>
-      <xacro:property name="imu_rpy" value="3.14 -1.57 0.0" lazy_eval="false"/>
-    </xacro:if>
-    <xacro:if value="${float(panther_version) > 1.06}">
+    <xacro:if value="${use_sim}">
       <xacro:property name="imu_xyz" value="-0.195 0.010 0.085" />
       <xacro:property name="imu_rpy" value="0.000 -0.000 3.142" />

Commit message: Fix imu tf frame (#373)
* Fix imu tf frame
* Reduce merge x y z  together
* Update panther_gazebo/launch/spawn_robot.launch.py

File: panther_description/urdf/panther.urdf.xacro (robot description, xacro)
@@ -5,10 +5,6 @@
   <!-- if lidars have to work correctly, use_gpu has to be true. -->
   <xacro:arg name="use_gpu" default="true" />
-  <xacro:arg name="imu_pos_x" default="0.169" />
-  <xacro:arg name="imu_pos_y" default="0.025" />
-  <xacro:arg name="imu_pos_z" default="0.092" />
-  <xacro:arg name="imu_rot_r" default="0.0" />
-  <xacro:arg name="imu_rot_p" default="0.0" />
-  <xacro:arg name="imu_rot_y" default="-1.57" />
+  <xacro:arg name="imu_xyz" default="0.169 0.025 0.092" />
+  <xacro:arg name="imu_rpy" default="0.0 0.0 -1.57" />
   <xacro:arg name="wheel_config_file"
     default="$(find panther_description)/config/WH01.yaml" />
@@ -22,10 +18,6 @@
     panther_version="$(arg panther_version)"
     use_sim="$(arg use_sim)"
-    imu_pos_x="$(arg imu_pos_x)"
-    imu_pos_y="$(arg imu_pos_y)"
-    imu_pos_z="$(arg imu_pos_z)"
-    imu_rot_r="$(arg imu_rot_r)"
-    imu_rot_p="$(arg imu_rot_p)"
-    imu_rot_y="$(arg imu_rot_y)"
+    imu_xyz="$(arg imu_xyz)"
+    imu_rpy="$(arg imu_rpy)"
     wheel_config_file="$(arg wheel_config_file)"
     controller_config_file="$(arg controller_config_file)"

File: panther_description/urdf/panther_macro.urdf.xacro (robot description, xacro)
@@ -8,11 +8,11 @@
             battery_config_file
             use_sim:=false
-            imu_pos_x:=0.168
-            imu_pos_y:=0.028
-            imu_pos_z:=0.083
-            imu_rot_r:=3.14
-            imu_rot_p:=-1.57
-            imu_rot_y:=0.0
+            imu_xyz:='0.169 0.025 0.092'
+            imu_rpy:='0.0 0.0 -1.57'
             namespace:=''">
+    <xacro:if value="${use_sim}">
+      <xacro:property name="imu_xyz" value="-0.195 0.010 0.085" />
+      <xacro:property name="imu_rpy" value="0.000 -0.000 3.142" />
+    </xacro:if>
     <xacro:if value="${namespace == ''}">
       <xacro:property name="ns" value="" />
@@ -30,10 +30,6 @@
     <xacro:body.body
       wheel_radius="${wheel_config['wheel_radius']}"
-      imu_pos_x="${imu_pos_x}"
-      imu_pos_y="${imu_pos_y}"
-      imu_pos_z="${imu_pos_z}"
-      imu_rot_r="${imu_rot_r}"
-      imu_rot_p="${imu_rot_p}"
-      imu_rot_y="${imu_rot_y}" />
+      imu_xyz="${imu_xyz}"
+      imu_rpy="${imu_rpy}" />
     <!-- WHEEL DECLARATION -->
     <xacro:wheel.wheel
