Commit message: Update body.urdf.xacro

File: panther_description/urdf/body.urdf.xacro (robot description, xacro)
@@ -26,5 +26,4 @@
       </collision>
       <inertial>
-        <origin xyz="-0.008 0.01 0.029" rpy="0.0 0.0 0.0"/>
         <mass value="43.0" />
         <inertia ixx="2.630036" ixy="-0.023480" ixz="0.052320"

Commit message: Update URDF to guide

File: panther_description/urdf/body.urdf.xacro (robot description, xacro)
@@ -7,5 +7,5 @@
     imu_rot_r imu_rot_p imu_rot_y" >
     <link name="base_link" />
-    <joint name="base_link_to_body_link_joint" type="fixed">
+    <joint name="base_to_body_joint" type="fixed">
       <origin xyz="0.0 0.0 ${wheel_radius}" rpy="0.0 0.0 0.0" />
       <parent link="base_link" />
@@ -14,16 +14,17 @@
     <link name="body_link">
       <visual>
+        <origin xyz="0.0 0.0 0.0" rpy="0.0 0.0 0.0"/>
         <geometry>
           <mesh filename="file://$(find panther_description)/meshes/body.dae" />
         </geometry>
-        <origin xyz="0.0 0.0 0.0" rpy="0.0 0.0 0.0"/>
       </visual>
       <collision>
+        <origin xyz="0.0 0.0 0.0" rpy="0.0 0.0 0.0"/>
         <geometry>
           <mesh filename="file://$(find panther_description)/meshes/body_collision.stl" />
         </geometry>
-        <origin xyz="0.0 0.0 0.0" rpy="0.0 0.0 0.0"/>
       </collision>
       <inertial>
+        <origin xyz="0.0 0.0 0.0" rpy="0.0 0.0 0.0" />
         <mass value="43.0" />
         <inertia ixx="2.630036" ixy="-0.023480" ixz="0.052320"
@@ -32,5 +33,5 @@
       </inertial>
     </link>
-    <joint name="body_link_to_imu_link_joint" type="fixed">
+    <joint name="body_to_imu_joint" type="fixed">
       <origin xyz="${imu_pos_x} ${imu_pos_y} ${imu_pos_z}"
               rpy="${imu_rot_r} ${imu_rot_p} ${imu_rot_y}" />
@@ -39,5 +40,5 @@
     </joint>
     <link name="imu_link" />
-    <joint name="body_link_front_light_link_joint" type="fixed">
+    <joint name="body_front_light_joint" type="fixed">
       <origin xyz="0.362 0.0 0.0" rpy="0.0 0.0 0.0" />
       <parent link="body_link" />
@@ -45,5 +46,5 @@
     </joint>
     <link name="front_light_link" />
-    <joint name="body_link_to_rear_light_link_joint" type="fixed">
+    <joint name="body_to_rear_light_joint" type="fixed">
       <origin xyz="-0.362 0.0 0.0" rpy="0.0 0.0 ${pi}" />
       <parent link="body_link" />
@@ -51,5 +52,5 @@
     </joint>
     <link name="rear_light_link" />
-    <joint name="body_link_to_cover_link_joint" type="fixed">
+    <joint name="body_to_cover_joint" type="fixed">
       <origin xyz="0.0 0.0 0.1715" rpy="0.0 0.0 0.0" />
       <parent link="body_link" />

File: panther_description/urdf/wheel.urdf.xacro (robot description, xacro)
@@ -24,7 +24,7 @@
     </xacro:if>
     <joint name="${prefix}_wheel_joint" type="continuous">
+      <origin xyz="${x} ${y} 0.0" rpy="0.0 0.0 0.0" />
       <parent link="body_link" />
       <child link="${prefix}_wheel_link" />
-      <origin xyz="${x} ${y} 0.0" rpy="0.0 0.0 0.0" />
       <axis xyz="0.0 1.0 0.0" />
       <limit effort="34.5" velocity="2.0" />
@@ -33,14 +33,14 @@
     <link name="${prefix}_wheel_link">
       <visual>
+        <origin xyz="0.0 0.0 0.0" rpy="0.0 0.0 0.0" />
         <geometry>
           <mesh filename="file://$(find ${wheel_config['mesh_package']})/${wheel_config['folder_path']}/${prefix}_wheel.dae" />
         </geometry>
-        <origin xyz="0.0 0.0 0.0" rpy="0.0 0.0 0.0" />
       </visual>
       <collision>
+        <origin xyz="0.0 0.0 0.0" rpy="0.0 0.0 0.0" />
         <geometry>
-          <mesh filename="file://$(find ${wheel_config['mesh_package']})/${wheel_config['folder_path']}/collision.stl" />
+          <mesh filename="file://$(find ${wheel_config['mesh_package']})/${wheel_config['folder_path']}/wheel_collision.stl" />
         </geometry>
-        <origin xyz="0.0 0.0 0.0" rpy="0.0 0.0 0.0" />
       </collision>
       <inertial>

Commit message: Update URDF to guide (#43)
* Update URDF to guide

* Remove unused node from launch

* Fix paths in README

* FIx wheel collision mesh name in README

* Add gazebo plugins dependency

* FIx joint name typo

File: panther_description/urdf/body.urdf.xacro (robot description, xacro)
@@ -7,5 +7,5 @@
     imu_rot_r imu_rot_p imu_rot_y" >
     <link name="base_link" />
-    <joint name="base_link_to_body_link_joint" type="fixed">
+    <joint name="base_to_body_joint" type="fixed">
       <origin xyz="0.0 0.0 ${wheel_radius}" rpy="0.0 0.0 0.0" />
       <parent link="base_link" />
@@ -14,16 +14,17 @@
     <link name="body_link">
       <visual>
+        <origin xyz="0.0 0.0 0.0" rpy="0.0 0.0 0.0"/>
         <geometry>
           <mesh filename="file://$(find panther_description)/meshes/body.dae" />
         </geometry>
-        <origin xyz="0.0 0.0 0.0" rpy="0.0 0.0 0.0"/>
       </visual>
       <collision>
+        <origin xyz="0.0 0.0 0.0" rpy="0.0 0.0 0.0"/>
         <geometry>
           <mesh filename="file://$(find panther_description)/meshes/body_collision.stl" />
         </geometry>
-        <origin xyz="0.0 0.0 0.0" rpy="0.0 0.0 0.0"/>
       </collision>
       <inertial>
+        <origin xyz="0.0 0.0 0.0" rpy="0.0 0.0 0.0" />
         <mass value="43.0" />
         <inertia ixx="2.630036" ixy="-0.023480" ixz="0.052320"
@@ -32,5 +33,5 @@
       </inertial>
     </link>
-    <joint name="body_link_to_imu_link_joint" type="fixed">
+    <joint name="body_to_imu_joint" type="fixed">
       <origin xyz="${imu_pos_x} ${imu_pos_y} ${imu_pos_z}"
               rpy="${imu_rot_r} ${imu_rot_p} ${imu_rot_y}" />
@@ -39,5 +40,5 @@
     </joint>
     <link name="imu_link" />
-    <joint name="body_link_front_light_link_joint" type="fixed">
+    <joint name="body_to_front_light_joint" type="fixed">
       <origin xyz="0.362 0.0 0.0" rpy="0.0 0.0 0.0" />
       <parent link="body_link" />
@@ -45,5 +46,5 @@
     </joint>
     <link name="front_light_link" />
-    <joint name="body_link_to_rear_light_link_joint" type="fixed">
+    <joint name="body_to_rear_light_joint" type="fixed">
       <origin xyz="-0.362 0.0 0.0" rpy="0.0 0.0 ${pi}" />
       <parent link="body_link" />
@@ -51,5 +52,5 @@
     </joint>
     <link name="rear_light_link" />
-    <joint name="body_link_to_cover_link_joint" type="fixed">
+    <joint name="body_to_cover_joint" type="fixed">
       <origin xyz="0.0 0.0 0.1715" rpy="0.0 0.0 0.0" />
       <parent link="body_link" />

Commit message: formatting

File: panther_description/urdf/body.urdf.xacro (robot description, xacro)
@@ -2,8 +2,10 @@
 <robot xmlns:xacro="http://www.ros.org/wiki/xacro">
   <!-- body defining macro -->
-  <xacro:macro name="body" params="
-    wheel_radius simulation_engine
-    imu_pos_x imu_pos_y imu_pos_z
-    imu_rot_r imu_rot_p imu_rot_y" >
+  <xacro:macro
+    name="body"
+    params="wheel_radius
+            simulation_engine
+            imu_pos_x imu_pos_y imu_pos_z
+            imu_rot_r imu_rot_p imu_rot_y">
     <link name="base_link" />
     <joint name="base_to_body_joint" type="fixed">
@@ -14,5 +16,5 @@
     <link name="body_link">
       <visual>
-        <origin xyz="0.0 0.0 0.0" rpy="0.0 0.0 0.0"/>
+        <origin xyz="0.0 0.0 0.0" rpy="0.0 0.0 0.0" />
         <geometry>
           <mesh filename="file://$(find panther_description)/meshes/body.dae" />
@@ -20,5 +22,5 @@
       </visual>
       <collision>
-        <origin xyz="0.0 0.0 0.0" rpy="0.0 0.0 0.0"/>
+        <origin xyz="0.0 0.0 0.0" rpy="0.0 0.0 0.0" />
         <geometry>
           <mesh filename="file://$(find panther_description)/meshes/body_collision.stl" />
@@ -35,5 +37,5 @@
     <joint name="body_to_imu_joint" type="fixed">
       <origin xyz="${imu_pos_x} ${imu_pos_y} ${imu_pos_z}"
-              rpy="${imu_rot_r} ${imu_rot_p} ${imu_rot_y}" />
+        rpy="${imu_rot_r} ${imu_rot_p} ${imu_rot_y}" />
       <parent link="body_link" />
       <child link="imu_link" />
@@ -60,6 +62,6 @@
     <xacro:if value="${simulation_engine == 'gazebo-classic'}">
       <!-- based on PhidgetSpatial datasheet -->
-      <xacro:property name="imu_acc_noise"  value="${280.0*1e-6*9.81}" />
-      <xacro:property name="imu_acc_drift"  value="${40.6*1e-6*9.81}" />
+      <xacro:property name="imu_acc_noise" value="${280.0*1e-6*9.81}" />
+      <xacro:property name="imu_acc_drift" value="${40.6*1e-6*9.81}" />
       <xacro:property name="imu_gyro_noise" value="${0.095*(pi/180.0)}" />
       <xacro:property name="imu_gyro_drift" value="${0.0042*(pi/180.0)}" />
@@ -76,5 +78,5 @@
         </plugin>
       </gazebo>
-  </xacro:if>
+    </xacro:if>
   </xacro:macro>
 </robot>

File: panther_description/urdf/components/external_antenna.urdf.xacro (robot description, xacro)
@@ -1,13 +1,14 @@
 <?xml version="1.0"?>
 <robot xmlns:xacro="http://www.ros.org/wiki/xacro">
-  <xacro:macro name="external_antenna"
-               params="parent_link xyz rpy
-                       tf_prefix:=None
-                       frame_id:=gps
-                       topic:=gps
-                       initial_latitude:=53.1978
-                       initial_longitude:=18.3735
-                       initial_altitude:=89.0
-                       simulation_engine:=gazebo-classic">
+  <xacro:macro
+    name="external_antenna"
+    params="parent_link xyz rpy
+            tf_prefix:=None
+            frame_id:=gps
+            topic:=gps
+            initial_latitude:=53.1978
+            initial_longitude:=18.3735
+            initial_altitude:=89.0
+            simulation_engine:=gazebo-classic">
     <xacro:if value="${tf_prefix == 'None'}">
       <xacro:property name="tf_prefix_ext" value="" />
@@ -23,5 +24,5 @@
     <link name="${tf_prefix_ext}external_antenna_link">
       <visual>
-        <origin xyz="0.0 0.0 0.0" rpy="0.0 0.0 0.0"/>
+        <origin xyz="0.0 0.0 0.0" rpy="0.0 0.0 0.0" />
         <geometry>
           <mesh filename="file://$(find panther_description)/meshes/components/external_antenna.dae" />
@@ -29,5 +30,5 @@
       </visual>
       <collision>
-        <origin xyz="0.0 0.0 0.0" rpy="0.0 0.0 0.0"/>
+        <origin xyz="0.0 0.0 0.0" rpy="0.0 0.0 0.0" />
         <geometry>
           <mesh filename="file://$(find panther_description)/meshes/components/external_antenna_collision.stl" />
@@ -35,5 +36,5 @@
       </collision>
       <inertial>
-        <origin xyz="0.045 0.0 0.0058" rpy="0.0 0.0 0.0"/>
+        <origin xyz="0.045 0.0 0.0058" rpy="0.0 0.0 0.0" />
         <mass value="0.59" />
         <inertia ixx="0.003964" ixy="0.0" ixz="0.0" iyy="0.0003964" iyz="0.0" izz="0.0004177" />

File: panther_description/urdf/panther.urdf.xacro (robot description, xacro)
@@ -1,3 +1,3 @@
-<?xml version='1.0'?>
+<?xml version="1.0" encoding="utf-8"?>
 <robot name="panther" xmlns:xacro="http://www.ros.org/wiki/xacro">
   <xacro:arg name="use_sim" default="false" />

File: panther_description/urdf/panther_macro.urdf.xacro (robot description, xacro)
@@ -1,16 +1,17 @@
 <?xml version='1.0'?>
 <robot xmlns:xacro="http://wiki.ros.org/xacro">
-  <xacro:macro name="panther_robot"
-               params="use_sim:=false
-                       dual_bat:=false
-                       imu_pos_x:=0.168
-                       imu_pos_y:=0.028
-                       imu_pos_z:=0.083
-                       imu_rot_r:=3.14
-                       imu_rot_p:=-1.57
-                       imu_rot_y:=0.0
-                       wheel_config_path:=None
-                       simulation_engine:='gazebo-classic'
-                       use_ros_control:=false">
+  <xacro:macro
+    name="panther_robot"
+    params="use_sim:=false
+            dual_bat:=false
+            imu_pos_x:=0.168
+            imu_pos_y:=0.028
+            imu_pos_z:=0.083
+            imu_rot_r:=3.14
+            imu_rot_p:=-1.57
+            imu_rot_y:=0.0
+            wheel_config_path:=None
+            simulation_engine:='gazebo-classic'
+            use_ros_control:=false">
     <xacro:if value="${wheel_config_path == 'None'}">
       <xacro:property name="wheel_config_file" value="$(find panther_description)/config/WH01.yaml" />

File: panther_description/urdf/wheel.urdf.xacro (robot description, xacro)
@@ -47,10 +47,11 @@
         <origin xyz="0.0 ${inertia_y_offset} 0.0" rpy="0.0 0.0 0.0" />
         <mass value="${wheel_config['mass']}" />
-        <inertia ixx="${wheel_config['inertia']['ixx']}"
-                 ixy="0.0"
-                 ixz="0.0"
-                 iyy="${wheel_config['inertia']['iyy']}"
-                 iyz="0.0"
-                 izz="${wheel_config['inertia']['izz']}" />
+        <inertia
+          ixx="${wheel_config['inertia']['ixx']}"
+          ixy="0.0"
+          ixz="0.0"
+          iyy="${wheel_config['inertia']['iyy']}"
+          iyz="0.0"
+          izz="${wheel_config['inertia']['izz']}" />
       </inertial>
     </link>

Commit message: code style cleanup

File: panther_description/urdf/body.urdf.xacro (robot description, xacro)
@@ -1,4 +1,4 @@
 <?xml version="1.0" encoding="utf-8"?>
-<robot xmlns:xacro="http://www.ros.org/wiki/xacro">
+<robot xmlns:xacro="http://wiki.ros.org/xacro">
   <!-- body defining macro -->
   <xacro:macro

File: panther_description/urdf/components/external_antenna.urdf.xacro (robot description, xacro)
@@ -1,4 +1,4 @@
-<?xml version="1.0"?>
-<robot xmlns:xacro="http://www.ros.org/wiki/xacro">
+<?xml version="1.0" encoding="utf-8"?>
+<robot xmlns:xacro="http://wiki.ros.org/xacro">
   <xacro:macro
     name="external_antenna"
@@ -38,5 +38,7 @@
         <origin xyz="0.045 0.0 0.0058" rpy="0.0 0.0 0.0" />
         <mass value="0.59" />
-        <inertia ixx="0.003964" ixy="0.0" ixz="0.0" iyy="0.0003964" iyz="0.0" izz="0.0004177" />
+        <inertia ixx="0.003964"  ixy="0.0"       ixz="0.0"
+                                 iyy="0.0003964" iyz="0.0"
+                                                 izz="0.0004177" />
       </inertial>
     </link>
@@ -50,5 +52,5 @@
     <gazebo>
       <plugin name="gps" filename="libhector_gazebo_ros_gps.so">
-        <updateRate>5</updateRate>
+        <updateRate>5.0</updateRate>
         <robotNamespace>/</robotNamespace>
         <bodyName>${tf_prefix_ext}${frame_id}</bodyName>

File: panther_description/urdf/panther.urdf.xacro (robot description, xacro)
@@ -1,4 +1,4 @@
 <?xml version="1.0" encoding="utf-8"?>
-<robot name="panther" xmlns:xacro="http://www.ros.org/wiki/xacro">
+<robot name="panther" xmlns:xacro="http://wiki.ros.org/xacro">
   <xacro:arg name="use_sim" default="false" />
   <xacro:arg name="use_gpu" default="false" />

File: panther_description/urdf/panther_macro.urdf.xacro (robot description, xacro)
@@ -1,3 +1,3 @@
-<?xml version='1.0'?>
+<?xml version="1.0" encoding="utf-8"?>
 <robot xmlns:xacro="http://wiki.ros.org/xacro">
   <xacro:macro

File: panther_description/urdf/wheel.urdf.xacro (robot description, xacro)
@@ -1,4 +1,4 @@
 <?xml version="1.0" encoding="utf-8"?>
-<robot xmlns:xacro="http://www.ros.org/wiki/xacro">
+<robot xmlns:xacro="http://wiki.ros.org/xacro">
   <!-- wheel defining macro -->
   <xacro:macro name="wheel" params="wheel_config wheel_separation_x hardware_interface prefix">

Commit message: Ros1 code style cleanup - KmakD (#81)
* formatting

* code style cleanup

* remove imu tf

File: panther_description/urdf/body.urdf.xacro (robot description, xacro)
@@ -1,9 +1,11 @@
 <?xml version="1.0" encoding="utf-8"?>
-<robot xmlns:xacro="http://www.ros.org/wiki/xacro">
+<robot xmlns:xacro="http://wiki.ros.org/xacro">
   <!-- body defining macro -->
-  <xacro:macro name="body" params="
-    wheel_radius simulation_engine
-    imu_pos_x imu_pos_y imu_pos_z
-    imu_rot_r imu_rot_p imu_rot_y" >
+  <xacro:macro
+    name="body"
+    params="wheel_radius
+            simulation_engine
+            imu_pos_x imu_pos_y imu_pos_z
+            imu_rot_r imu_rot_p imu_rot_y">
     <link name="base_link" />
     <joint name="base_to_body_joint" type="fixed">
@@ -14,5 +16,5 @@
     <link name="body_link">
       <visual>
-        <origin xyz="0.0 0.0 0.0" rpy="0.0 0.0 0.0"/>
+        <origin xyz="0.0 0.0 0.0" rpy="0.0 0.0 0.0" />
         <geometry>
           <mesh filename="file://$(find panther_description)/meshes/body.dae" />
@@ -20,5 +22,5 @@
       </visual>
       <collision>
-        <origin xyz="0.0 0.0 0.0" rpy="0.0 0.0 0.0"/>
+        <origin xyz="0.0 0.0 0.0" rpy="0.0 0.0 0.0" />
         <geometry>
           <mesh filename="file://$(find panther_description)/meshes/body_collision.stl" />
@@ -35,5 +37,5 @@
     <joint name="body_to_imu_joint" type="fixed">
       <origin xyz="${imu_pos_x} ${imu_pos_y} ${imu_pos_z}"
-              rpy="${imu_rot_r} ${imu_rot_p} ${imu_rot_y}" />
+        rpy="${imu_rot_r} ${imu_rot_p} ${imu_rot_y}" />
       <parent link="body_link" />
       <child link="imu_link" />
@@ -60,6 +62,6 @@
     <xacro:if value="${simulation_engine == 'gazebo-classic'}">
       <!-- based on PhidgetSpatial datasheet -->
-      <xacro:property name="imu_acc_noise"  value="${280.0*1e-6*9.81}" />
-      <xacro:property name="imu_acc_drift"  value="${40.6*1e-6*9.81}" />
+      <xacro:property name="imu_acc_noise" value="${280.0*1e-6*9.81}" />
+      <xacro:property name="imu_acc_drift" value="${40.6*1e-6*9.81}" />
       <xacro:property name="imu_gyro_noise" value="${0.095*(pi/180.0)}" />
       <xacro:property name="imu_gyro_drift" value="${0.0042*(pi/180.0)}" />
@@ -76,5 +78,5 @@
         </plugin>
       </gazebo>
-  </xacro:if>
+    </xacro:if>
   </xacro:macro>
 </robot>

File: panther_description/urdf/components/external_antenna.urdf.xacro (robot description, xacro)
@@ -1,13 +1,14 @@
-<?xml version="1.0"?>
-<robot xmlns:xacro="http://www.ros.org/wiki/xacro">
-  <xacro:macro name="external_antenna"
-               params="parent_link xyz rpy
-                       tf_prefix:=None
-                       frame_id:=gps
-                       topic:=gps
-                       initial_latitude:=53.1978
-                       initial_longitude:=18.3735
-                       initial_altitude:=89.0
-                       simulation_engine:=gazebo-classic">
+<?xml version="1.0" encoding="utf-8"?>
+<robot xmlns:xacro="http://wiki.ros.org/xacro">
+  <xacro:macro
+    name="external_antenna"
+    params="parent_link xyz rpy
+            tf_prefix:=None
+            frame_id:=gps
+            topic:=gps
+            initial_latitude:=53.1978
+            initial_longitude:=18.3735
+            initial_altitude:=89.0
+            simulation_engine:=gazebo-classic">
     <xacro:if value="${tf_prefix == 'None'}">
       <xacro:property name="tf_prefix_ext" value="" />
@@ -23,5 +24,5 @@
     <link name="${tf_prefix_ext}external_antenna_link">
       <visual>
-        <origin xyz="0.0 0.0 0.0" rpy="0.0 0.0 0.0"/>
+        <origin xyz="0.0 0.0 0.0" rpy="0.0 0.0 0.0" />
         <geometry>
           <mesh filename="file://$(find panther_description)/meshes/components/external_antenna.dae" />
@@ -29,5 +30,5 @@
       </visual>
       <collision>
-        <origin xyz="0.0 0.0 0.0" rpy="0.0 0.0 0.0"/>
+        <origin xyz="0.0 0.0 0.0" rpy="0.0 0.0 0.0" />
         <geometry>
           <mesh filename="file://$(find panther_description)/meshes/components/external_antenna_collision.stl" />
@@ -35,7 +36,9 @@
       </collision>
       <inertial>
-        <origin xyz="0.045 0.0 0.0058" rpy="0.0 0.0 0.0"/>
+        <origin xyz="0.045 0.0 0.0058" rpy="0.0 0.0 0.0" />
         <mass value="0.59" />
-        <inertia ixx="0.003964" ixy="0.0" ixz="0.0" iyy="0.0003964" iyz="0.0" izz="0.0004177" />
+        <inertia ixx="0.003964"  ixy="0.0"       ixz="0.0"
+                                 iyy="0.0003964" iyz="0.0"
+                                                 izz="0.0004177" />
       </inertial>
     </link>
@@ -49,5 +52,5 @@
     <gazebo>
       <plugin name="gps" filename="libhector_gazebo_ros_gps.so">
-        <updateRate>5</updateRate>
+        <updateRate>5.0</updateRate>
         <robotNamespace>/</robotNamespace>
         <bodyName>${tf_prefix_ext}${frame_id}</bodyName>

File: panther_description/urdf/panther.urdf.xacro (robot description, xacro)
@@ -1,4 +1,4 @@
-<?xml version='1.0'?>
-<robot name="panther" xmlns:xacro="http://www.ros.org/wiki/xacro">
+<?xml version="1.0" encoding="utf-8"?>
+<robot name="panther" xmlns:xacro="http://wiki.ros.org/xacro">
   <xacro:arg name="use_sim" default="false" />
   <xacro:arg name="use_gpu" default="false" />

File: panther_description/urdf/panther_macro.urdf.xacro (robot description, xacro)
@@ -1,16 +1,17 @@
-<?xml version='1.0'?>
+<?xml version="1.0" encoding="utf-8"?>
 <robot xmlns:xacro="http://wiki.ros.org/xacro">
-  <xacro:macro name="panther_robot"
-               params="use_sim:=false
-                       dual_bat:=false
-                       imu_pos_x:=0.168
-                       imu_pos_y:=0.028
-                       imu_pos_z:=0.083
-                       imu_rot_r:=3.14
-                       imu_rot_p:=-1.57
-                       imu_rot_y:=0.0
-                       wheel_config_path:=None
-                       simulation_engine:='gazebo-classic'
-                       use_ros_control:=false">
+  <xacro:macro
+    name="panther_robot"
+    params="use_sim:=false
+            dual_bat:=false
+            imu_pos_x:=0.168
+            imu_pos_y:=0.028
+            imu_pos_z:=0.083
+            imu_rot_r:=3.14
+            imu_rot_p:=-1.57
+            imu_rot_y:=0.0
+            wheel_config_path:=None
+            simulation_engine:='gazebo-classic'
+            use_ros_control:=false">
     <xacro:if value="${wheel_config_path == 'None'}">
       <xacro:property name="wheel_config_file" value="$(find panther_description)/config/WH01.yaml" />

File: panther_description/urdf/wheel.urdf.xacro (robot description, xacro)
@@ -1,4 +1,4 @@
 <?xml version="1.0" encoding="utf-8"?>
-<robot xmlns:xacro="http://www.ros.org/wiki/xacro">
+<robot xmlns:xacro="http://wiki.ros.org/xacro">
   <!-- wheel defining macro -->
   <xacro:macro name="wheel" params="wheel_config wheel_separation_x hardware_interface prefix">
@@ -47,10 +47,11 @@
         <origin xyz="0.0 ${inertia_y_offset} 0.0" rpy="0.0 0.0 0.0" />
         <mass value="${wheel_config['mass']}" />
-        <inertia ixx="${wheel_config['inertia']['ixx']}"
-                 ixy="0.0"
-                 ixz="0.0"
-                 iyy="${wheel_config['inertia']['iyy']}"
-                 iyz="0.0"
-                 izz="${wheel_config['inertia']['izz']}" />
+        <inertia
+          ixx="${wheel_config['inertia']['ixx']}"
+          ixy="0.0"
+          ixz="0.0"
+          iyy="${wheel_config['inertia']['iyy']}"
+          iyz="0.0"
+          izz="${wheel_config['inertia']['izz']}" />
       </inertial>
     </link>
