Commit message: basic plugin usage - POC

File: panther_description/urdf/body.urdf.xacro (robot description, xacro)
@@ -48,4 +48,10 @@
     </joint>
     <link name="front_light_link" />
+    <joint name="front_light_to_front_animation_joint" type="fixed">
+      <origin xyz="0.0 0.0 0.0185" rpy="${pi/2} 0.0 ${pi/2}" />
+      <parent link="front_light_link" />
+      <child link="front_animation_link" />
+    </joint>
+    <link name="front_animation_link" />
     <joint name="body_to_rear_light_joint" type="fixed">
       <origin xyz="-0.362 0.0 0.0" rpy="0.0 0.0 ${pi}" />

Commit message: add rear animation texture

File: panther_description/urdf/body.urdf.xacro (robot description, xacro)
@@ -60,4 +60,10 @@
     </joint>
     <link name="rear_light_link" />
+    <joint name="rear_light_to_rear_animation_joint" type="fixed">
+      <origin xyz="0.0 0.0 0.0185" rpy="${pi/2} 0.0 ${pi/2}" />
+      <parent link="rear_light_link" />
+      <child link="rear_animation_link" />
+    </joint>
+    <link name="rear_animation_link" />
     <joint name="body_to_cover_joint" type="fixed">
       <origin xyz="0.0 0.0 0.1715" rpy="0.0 0.0 0.0" />

Commit message: Rviz lights plugin (#111)
* basic plugin usage - POC

* add rear animation texture

* fix rviz config

* fix .rviz file

File: panther_description/urdf/body.urdf.xacro (robot description, xacro)
@@ -48,4 +48,10 @@
     </joint>
     <link name="front_light_link" />
+    <joint name="front_light_to_front_animation_joint" type="fixed">
+      <origin xyz="0.0 0.0 0.0185" rpy="${pi/2} 0.0 ${pi/2}" />
+      <parent link="front_light_link" />
+      <child link="front_animation_link" />
+    </joint>
+    <link name="front_animation_link" />
     <joint name="body_to_rear_light_joint" type="fixed">
       <origin xyz="-0.362 0.0 0.0" rpy="0.0 0.0 ${pi}" />
@@ -54,4 +60,10 @@
     </joint>
     <link name="rear_light_link" />
+    <joint name="rear_light_to_rear_animation_joint" type="fixed">
+      <origin xyz="0.0 0.0 0.0185" rpy="${pi/2} 0.0 ${pi/2}" />
+      <parent link="rear_light_link" />
+      <child link="rear_animation_link" />
+    </joint>
+    <link name="rear_animation_link" />
     <joint name="body_to_cover_joint" type="fixed">
       <origin xyz="0.0 0.0 0.1715" rpy="0.0 0.0 0.0" />

Commit message: Rename light_link to bumper_link

File: panther_description/urdf/body.urdf.xacro (robot description, xacro)
@@ -42,28 +42,28 @@
     </joint>
     <link name="imu_link" />
-    <joint name="body_to_front_light_joint" type="fixed">
+    <joint name="body_to_front_bumper_joint" type="fixed">
       <origin xyz="0.362 0.0 0.0" rpy="0.0 0.0 0.0" />
       <parent link="body_link" />
+      <child link="front_bumper_link" />
+    </joint>
+    <link name="front_bumper_link" />
+    <joint name="front_bumper_to_front_light_joint" type="fixed">
+      <origin xyz="0.0 0.0 0.0185" rpy="${pi/2} 0.0 ${pi/2}" />
+      <parent link="front_bumper_link" />
       <child link="front_light_link" />
     </joint>
     <link name="front_light_link" />
-    <joint name="front_light_to_front_animation_joint" type="fixed">
-      <origin xyz="0.0 0.0 0.0185" rpy="${pi/2} 0.0 ${pi/2}" />
-      <parent link="front_light_link" />
-      <child link="front_animation_link" />
-    </joint>
-    <link name="front_animation_link" />
-    <joint name="body_to_rear_light_joint" type="fixed">
+    <joint name="body_to_rear_bumper_joint" type="fixed">
       <origin xyz="-0.362 0.0 0.0" rpy="0.0 0.0 ${pi}" />
       <parent link="body_link" />
+      <child link="rear_bumper_link" />
+    </joint>
+    <link name="rear_bumper_link" />
+    <joint name="rear_bumper_to_rear_light_joint" type="fixed">
+      <origin xyz="0.0 0.0 0.0185" rpy="${pi/2} 0.0 ${pi/2}" />
+      <parent link="rear_bumper_link" />
       <child link="rear_light_link" />
     </joint>
     <link name="rear_light_link" />
-    <joint name="rear_light_to_rear_animation_joint" type="fixed">
-      <origin xyz="0.0 0.0 0.0185" rpy="${pi/2} 0.0 ${pi/2}" />
-      <parent link="rear_light_link" />
-      <child link="rear_animation_link" />
-    </joint>
-    <link name="rear_animation_link" />
     <joint name="body_to_cover_joint" type="fixed">
       <origin xyz="0.0 0.0 0.1715" rpy="0.0 0.0 0.0" />

Commit message: Change finding mesh files method

File: panther_description/urdf/body.urdf.xacro (robot description, xacro)
@@ -18,5 +18,5 @@
         <origin xyz="0.0 0.0 0.0" rpy="0.0 0.0 0.0" />
         <geometry>
-          <mesh filename="file://$(find panther_description)/meshes/body.dae" />
+          <mesh filename="package://panther_description/meshes/body.dae" />
         </geometry>
       </visual>
@@ -24,5 +24,5 @@
         <origin xyz="0.0 0.0 0.0" rpy="0.0 0.0 0.0" />
         <geometry>
-          <mesh filename="file://$(find panther_description)/meshes/body_collision.stl" />
+          <mesh filename="package://panther_description/meshes/body_collision.stl" />
         </geometry>
       </collision>

File: panther_description/urdf/components/external_antenna.urdf.xacro (robot description, xacro)
@@ -26,5 +26,5 @@
         <origin xyz="0.0 0.0 0.0" rpy="0.0 0.0 0.0" />
         <geometry>
-          <mesh filename="file://$(find panther_description)/meshes/components/external_antenna.dae" />
+          <mesh filename="package://panther_description/meshes/components/external_antenna.dae" />
         </geometry>
       </visual>
@@ -32,5 +32,5 @@
         <origin xyz="0.0 0.0 0.0" rpy="0.0 0.0 0.0" />
         <geometry>
-          <mesh filename="file://$(find panther_description)/meshes/components/external_antenna_collision.stl" />
+          <mesh filename="package://panther_description/meshes/components/external_antenna_collision.stl" />
         </geometry>
       </collision>

File: panther_description/urdf/wheel.urdf.xacro (robot description, xacro)
@@ -35,5 +35,5 @@
         <origin xyz="0.0 0.0 0.0" rpy="0.0 0.0 0.0" />
         <geometry>
-          <mesh filename="file://$(find ${wheel_config['mesh_package']})/${wheel_config['folder_path']}/${prefix}_wheel.dae" />
+          <mesh filename="package://${wheel_config['mesh_package']}/${wheel_config['folder_path']}/${prefix}_wheel.dae" />
         </geometry>
       </visual>
@@ -41,5 +41,5 @@
         <origin xyz="0.0 0.0 0.0" rpy="0.0 0.0 0.0" />
         <geometry>
-          <mesh filename="file://$(find ${wheel_config['mesh_package']})/${wheel_config['folder_path']}/wheel_collision.stl" />
+          <mesh filename="package://${wheel_config['mesh_package']}/${wheel_config['folder_path']}/wheel_collision.stl" />
         </geometry>
       </collision>

Commit message: Second option

File: panther_description/urdf/body.urdf.xacro (robot description, xacro)
@@ -4,20 +4,14 @@
   <xacro:macro
     name="body"
-    params="namespace wheel_radius
+    params="wheel_radius
             imu_pos_x imu_pos_y imu_pos_z
             imu_rot_r imu_rot_p imu_rot_y">
-    <xacro:if value="${namespace == ''}">
-      <xacro:property name="ns" value="" />
-    </xacro:if>
-    <xacro:unless value="${namespace == ''}">
-        <xacro:property name="ns" value="${namespace}/" />
-    </xacro:unless>
-    <link name="${ns}base_link" />
+    <link name="base_link" />
     <joint name="base_to_body_joint" type="fixed">
       <origin xyz="0.0 0.0 ${wheel_radius}" rpy="0.0 0.0 0.0" />
-      <parent link="${ns}base_link" />
-      <child link="${ns}body_link" />
+      <parent link="base_link" />
+      <child link="body_link" />
     </joint>
-    <link name="${ns}body_link">
+    <link name="body_link">
       <visual>
         <origin xyz="0.0 0.0 0.0" rpy="0.0 0.0 0.0" />
@@ -43,38 +37,38 @@
       <origin xyz="${imu_pos_x} ${imu_pos_y} ${imu_pos_z}"
         rpy="${imu_rot_r} ${imu_rot_p} ${imu_rot_y}" />
-      <parent link="${ns}body_link" />
-      <child link="${ns}imu_link" />
+      <parent link="body_link" />
+      <child link="imu_link" />
     </joint>
-    <link name="${ns}imu_link" />
+    <link name="imu_link" />
     <joint name="body_to_front_bumper_joint" type="fixed">
       <origin xyz="0.362 0.0 0.0" rpy="0.0 0.0 0.0" />
-      <parent link="${ns}body_link" />
-      <child link="${ns}front_bumper_link" />
+      <parent link="body_link" />
+      <child link="front_bumper_link" />
     </joint>
-    <link name="${ns}front_bumper_link" />
+    <link name="front_bumper_link" />
     <joint name="front_bumper_to_front_light_joint" type="fixed">
       <origin xyz="0.0 0.0 0.0185" rpy="${pi/2} 0.0 ${pi/2}" />
-      <parent link="${ns}front_bumper_link" />
-      <child link="${ns}front_light_link" />
+      <parent link="front_bumper_link" />
+      <child link="front_light_link" />
     </joint>
-    <link name="${ns}front_light_link" />
+    <link name="front_light_link" />
     <joint name="body_to_rear_bumper_joint" type="fixed">
       <origin xyz="-0.362 0.0 0.0" rpy="0.0 0.0 ${pi}" />
-      <parent link="${ns}body_link" />
-      <child link="${ns}rear_bumper_link" />
+      <parent link="body_link" />
+      <child link="rear_bumper_link" />
     </joint>
-    <link name="${ns}rear_bumper_link" />
+    <link name="rear_bumper_link" />
     <joint name="rear_bumper_to_rear_light_joint" type="fixed">
       <origin xyz="0.0 0.0 0.0185" rpy="${pi/2} 0.0 ${pi/2}" />
-      <parent link="${ns}rear_bumper_link" />
-      <child link="${ns}rear_light_link" />
+      <parent link="rear_bumper_link" />
+      <child link="rear_light_link" />
     </joint>
-    <link name="${ns}rear_light_link" />
+    <link name="rear_light_link" />
     <joint name="body_to_cover_joint" type="fixed">
       <origin xyz="0.0 0.0 0.1715" rpy="0.0 0.0 0.0" />
-      <parent link="${ns}body_link" />
-      <child link="${ns}cover_link" />
+      <parent link="body_link" />
+      <child link="cover_link" />
     </joint>
-    <link name="${ns}cover_link" />
+    <link name="cover_link" />
   </xacro:macro>
 </robot>

File: panther_description/urdf/panther_macro.urdf.xacro (robot description, xacro)
@@ -30,5 +30,4 @@
     <!-- BODY DECLARATION -->
     <xacro:body.body
-      namespace="${namespace}"
       wheel_radius="${wheel_config['wheel_radius']}"
       imu_pos_x="${imu_pos_x}"
@@ -40,20 +39,16 @@
     <!-- WHEEL DECLARATION -->
     <xacro:wheel.wheel
-      namespace="${namespace}"
       wheel_config="${wheel_config}"
       wheel_separation_x="${wheel_separation_x}"
       prefix="fl" />
     <xacro:wheel.wheel
-      namespace="${namespace}"
       wheel_config="${wheel_config}"
       wheel_separation_x="${wheel_separation_x}"
       prefix="fr" />
     <xacro:wheel.wheel
-      namespace="${namespace}"
       wheel_config="${wheel_config}"
       wheel_separation_x="${wheel_separation_x}"
       prefix="rl" />
     <xacro:wheel.wheel
-      namespace="${namespace}"
       wheel_config="${wheel_config}"
       wheel_separation_x="${wheel_separation_x}"
@@ -171,5 +166,5 @@
       <xacro:gazebo.battery config_file="${battery_config_file}" namespace="${namespace}" />
       <xacro:gazebo.controller config_file="${controller_config_file}" namespace="${namespace}" />
-      <xacro:gazebo.imu reference_frame="${ns}imu_link" namespace="${namespace}" />
+      <xacro:gazebo.imu reference_frame="imu_link" namespace="${namespace}" />
     </xacro:if>
   </xacro:macro>

File: panther_description/urdf/wheel.urdf.xacro (robot description, xacro)
@@ -2,11 +2,5 @@
 <robot xmlns:xacro="http://wiki.ros.org/xacro">
   <!-- wheel defining macro -->
-  <xacro:macro name="wheel" params="namespace wheel_config wheel_separation_x prefix">
-  <xacro:if value="${namespace == ''}">
-    <xacro:property name="ns" value="" />
-  </xacro:if>
-  <xacro:unless value="${namespace == ''}">
-      <xacro:property name="ns" value="${namespace}/" />
-  </xacro:unless>
+  <xacro:macro name="wheel" params="wheel_config wheel_separation_x prefix">
     <xacro:if value="${prefix == 'fl'}">
       <xacro:property name="x" value="${wheel_separation_x/2.0}" />
@@ -35,11 +29,11 @@
     <joint name="${prefix}_wheel_joint" type="continuous">
       <origin xyz="${x} ${y} 0.0" rpy="0.0 0.0 0.0" />
-      <parent link="${ns}body_link" />
-      <child link="${ns}${prefix}_wheel_link" />
+      <parent link="body_link" />
+      <child link="${prefix}_wheel_link" />
       <axis xyz="0.0 1.0 0.0" />
       <limit effort="64.5" velocity="10.958" />
       <dynamics damping="0.01" friction="0.1" />
     </joint>
-    <link name="${ns}${prefix}_wheel_link">
+    <link name="${prefix}_wheel_link">
       <visual>
         <origin xyz="0.0 0.0 0.0" rpy="0.0 0.0 0.0" />
@@ -68,5 +62,5 @@
     </link>
     <xacro:if value="${use_sim}">
-      <gazebo reference="${ns}${prefix}_wheel_link" xmlns:ignition="http://ignitionrobotics.org/schema">
+      <gazebo reference="${prefix}_wheel_link" xmlns:ignition="http://ignitionrobotics.org/schema">
         <collision>
           <surface>
@@ -75,5 +69,5 @@
                 <mu>1.0</mu>
                 <mu2>0.0</mu2>
-                <fdir1 ignition:expressed_in="${ns}base_link">${fdir}</fdir1>
+                <fdir1 ignition:expressed_in="base_link">${fdir}</fdir1>
               </ode>
             </friction>

Commit message: Add lights to urdf

File: panther_description/urdf/body.urdf.xacro (robot description, xacro)
@@ -48,5 +48,5 @@
     <link name="front_bumper_link" />
     <joint name="front_bumper_to_front_light_joint" type="fixed">
-      <origin xyz="0.0 0.0 0.0185" rpy="${pi/2} 0.0 ${pi/2}" />
+      <origin xyz="0.0 0.0 0.0185" rpy="0.0 -${pi/2} 0.0" />
       <parent link="front_bumper_link" />
       <child link="front_light_link" />
@@ -60,5 +60,5 @@
     <link name="rear_bumper_link" />
     <joint name="rear_bumper_to_rear_light_joint" type="fixed">
-      <origin xyz="0.0 0.0 0.0185" rpy="${pi/2} 0.0 ${pi/2}" />
+      <origin xyz="0.0 0.0 0.0185" rpy="0.0 -${pi/2} 0.0" />
       <parent link="rear_bumper_link" />
       <child link="rear_light_link" />
@@ -71,4 +71,32 @@
     </joint>
     <link name="cover_link" />
+    <gazebo reference="front_light_link">
+      <light name="panther_front_light" type="spot">
+        <cast_shadows>false</cast_shadows>
+        <visualize>0</visualize>
+        <diffuse>1.0 1.0 1.0</diffuse>
+        <specular>1.0 1.0 1.0</specular>
+        <direction>0 0 -1</direction>
+        <intensity>1.0</intensity>
+        <spot>
+          <inner_angle>2.1</inner_angle>
+          <outer_angle>2.1</outer_angle>
+        </spot>
+      </light>
+    </gazebo>
+    <gazebo reference="rear_light_link">
+      <light name="panther_rear_light" type="spot">
+        <cast_shadows>false</cast_shadows>
+        <visualize>0</visualize>
+        <diffuse>1.0 1.0 1.0</diffuse>
+        <specular>1.0 1.0 1.0</specular>
+        <direction>0 0 -1</direction>
+        <intensity>1.0</intensity>
+        <spot>
+          <inner_angle>2.1</inner_angle>
+          <outer_angle>2.1</outer_angle>
+        </spot>
+      </light>
+    </gazebo>
   </xacro:macro>
 </robot>

Commit message: Add light macro

File: panther_description/urdf/body.urdf.xacro (robot description, xacro)
@@ -42,5 +42,5 @@
     <link name="imu_link" />
     <joint name="body_to_front_bumper_joint" type="fixed">
-      <origin xyz="0.362 0.0 0.0" rpy="0.0 0.0 0.0" />
+      <origin xyz="0.36 0.0 0.0" rpy="0.0 0.0 0.0" />
       <parent link="body_link" />
       <child link="front_bumper_link" />
@@ -48,11 +48,20 @@
     <link name="front_bumper_link" />
     <joint name="front_bumper_to_front_light_joint" type="fixed">
-      <origin xyz="0.0 0.0 0.0185" rpy="0.0 -${pi/2} 0.0" />
+      <origin xyz="0.0 0.0 0.0185" rpy="0.0 0.0 0.0" />
       <parent link="front_bumper_link" />
       <child link="front_light_link" />
     </joint>
-    <link name="front_light_link" />
+    <link name="front_light_link">
+      <visual name="front_light_vis">
+        <geometry>
+          <box size="0.005 0.5 0.015"/>
+        </geometry>
+        <material name="white">
+          <color rgba="1 1 1 1"/>
+        </material>
+      </visual>
+    </link>
     <joint name="body_to_rear_bumper_joint" type="fixed">
-      <origin xyz="-0.362 0.0 0.0" rpy="0.0 0.0 ${pi}" />
+      <origin xyz="-0.36 0.0 0.0" rpy="0.0 0.0 ${pi}" />
       <parent link="body_link" />
       <child link="rear_bumper_link" />
@@ -60,9 +69,18 @@
     <link name="rear_bumper_link" />
     <joint name="rear_bumper_to_rear_light_joint" type="fixed">
-      <origin xyz="0.0 0.0 0.0185" rpy="0.0 -${pi/2} 0.0" />
+      <origin xyz="0.0 0.0 0.0185" rpy="0.0 0.0 0.0" />
       <parent link="rear_bumper_link" />
       <child link="rear_light_link" />
     </joint>
-    <link name="rear_light_link" />
+    <link name="rear_light_link">
+      <visual name="rear_light_vis">
+        <geometry>
+          <box size="0.005 0.5 0.015"/>
+        </geometry>
+        <material name="white">
+          <color rgba="1 1 1 1"/>
+        </material>
+      </visual>
+    </link>
     <joint name="body_to_cover_joint" type="fixed">
       <origin xyz="0.0 0.0 0.1715" rpy="0.0 0.0 0.0" />
@@ -71,32 +89,4 @@
     </joint>
     <link name="cover_link" />
-    <gazebo reference="front_light_link">
-      <light name="panther_front_light" type="spot">
-        <cast_shadows>false</cast_shadows>
-        <visualize>0</visualize>
-        <diffuse>1.0 1.0 1.0</diffuse>
-        <specular>1.0 1.0 1.0</specular>
-        <direction>0 0 -1</direction>
-        <intensity>1.0</intensity>
-        <spot>
-          <inner_angle>2.1</inner_angle>
-          <outer_angle>2.1</outer_angle>
-        </spot>
-      </light>
-    </gazebo>
-    <gazebo reference="rear_light_link">
-      <light name="panther_rear_light" type="spot">
-        <cast_shadows>false</cast_shadows>
-        <visualize>0</visualize>
-        <diffuse>1.0 1.0 1.0</diffuse>
-        <specular>1.0 1.0 1.0</specular>
-        <direction>0 0 -1</direction>
-        <intensity>1.0</intensity>
-        <spot>
-          <inner_angle>2.1</inner_angle>
-          <outer_angle>2.1</outer_angle>
-        </spot>
-      </light>
-    </gazebo>
   </xacro:macro>
 </robot>

File: panther_description/urdf/gazebo.urdf.xacro (robot description, xacro)
@@ -15,5 +15,5 @@
       <plugin filename="ignition-gazebo-linearbatteryplugin-system"
         name="gz::sim::systems::LinearBatteryPlugin">
-        <battery_name>${ns}panther_battery</battery_name>
+        <battery_name>${ns}battery</battery_name>
         <voltage>41.4</voltage>
         <open_circuit_voltage_constant_coef>42.0</open_circuit_voltage_constant_coef>
@@ -106,3 +106,20 @@
     </gazebo>
   </xacro:macro>
+  <!-- Lights -->
+  <xacro:macro name="light" params="reference_frame name namespace:=''">
+    <gazebo reference="${reference_frame}">
+      <light name="${name}" type="spot">
+        <cast_shadows>false</cast_shadows>
+        <visualize>0</visualize>
+        <diffuse>1.0 1.0 1.0</diffuse>
+        <specular>1.0 1.0 1.0</specular>
+        <direction>1 0 0</direction>
+        <intensity>1.0</intensity>
+        <spot>
+          <inner_angle>2.1</inner_angle>
+          <outer_angle>2.1</outer_angle>
+        </spot>
+      </light>
+    </gazebo>
+  </xacro:macro>
 </robot>

File: panther_description/urdf/panther_macro.urdf.xacro (robot description, xacro)
@@ -167,4 +167,6 @@
       <xacro:gazebo.controller config_file="${controller_config_file}" namespace="${namespace}" />
       <xacro:gazebo.imu reference_frame="imu_link" namespace="${namespace}" />
+      <xacro:gazebo.light reference_frame="front_light_link" name="front_light" namespace="${namespace}" />
+      <xacro:gazebo.light reference_frame="rear_light_link" name="rear_light" namespace="${namespace}" />
     </xacro:if>
   </xacro:macro>

Commit message: Steering lights from channel topics

File: panther_description/urdf/body.urdf.xacro (robot description, xacro)
@@ -42,5 +42,5 @@
     <link name="imu_link" />
     <joint name="body_to_front_bumper_joint" type="fixed">
-      <origin xyz="0.36 0.0 0.0" rpy="0.0 0.0 0.0" />
+      <origin xyz="0.363 0.0 0.0" rpy="0.0 0.0 0.0" />
       <parent link="body_link" />
       <child link="front_bumper_link" />
@@ -54,6 +54,7 @@
     <link name="front_light_link">
       <visual name="front_light_vis">
+        <cast_shadows>false</cast_shadows>
         <geometry>
-          <box size="0.005 0.5 0.015"/>
+          <box size="0.001 0.5 0.015"/>
         </geometry>
         <material name="white">
@@ -63,5 +64,5 @@
     </link>
     <joint name="body_to_rear_bumper_joint" type="fixed">
-      <origin xyz="-0.36 0.0 0.0" rpy="0.0 0.0 ${pi}" />
+      <origin xyz="-0.363 0.0 0.0" rpy="0.0 0.0 ${pi}" />
       <parent link="body_link" />
       <child link="rear_bumper_link" />
@@ -75,6 +76,7 @@
     <link name="rear_light_link">
       <visual name="rear_light_vis">
+        <cast_shadows>false</cast_shadows>
         <geometry>
-          <box size="0.005 0.5 0.015"/>
+          <box size="0.001 0.5 0.015"/>
         </geometry>
         <material name="white">

File: panther_description/urdf/gazebo.urdf.xacro (robot description, xacro)
@@ -110,5 +110,5 @@
     <gazebo reference="${reference_frame}">
       <light name="${name}" type="spot">
-        <cast_shadows>false</cast_shadows>
+        <cast_shadows>true</cast_shadows>
         <visualize>0</visualize>
         <diffuse>1.0 1.0 1.0</diffuse>
@@ -117,6 +117,7 @@
         <intensity>1.0</intensity>
         <spot>
-          <inner_angle>2.1</inner_angle>
-          <outer_angle>2.1</outer_angle>
+          <inner_angle>1.0</inner_angle>
+          <outer_angle>2.0</outer_angle>
+          <falloff>0.4</falloff>
         </spot>
       </light>

Commit message: Simplify and add cmd_vel

File: panther_description/urdf/body.urdf.xacro (robot description, xacro)
@@ -52,15 +52,5 @@
       <child link="front_light_link" />
     </joint>
-    <link name="front_light_link">
-      <visual name="front_light_vis">
-        <cast_shadows>false</cast_shadows>
-        <geometry>
-          <box size="0.001 0.5 0.015"/>
-        </geometry>
-        <material name="white">
-          <color rgba="1 1 1 1"/>
-        </material>
-      </visual>
-    </link>
+    <link name="front_light_link"/>
     <joint name="body_to_rear_bumper_joint" type="fixed">
       <origin xyz="-0.363 0.0 0.0" rpy="0.0 0.0 ${pi}" />
@@ -74,15 +64,5 @@
       <child link="rear_light_link" />
     </joint>
-    <link name="rear_light_link">
-      <visual name="rear_light_vis">
-        <cast_shadows>false</cast_shadows>
-        <geometry>
-          <box size="0.001 0.5 0.015"/>
-        </geometry>
-        <material name="white">
-          <color rgba="1 1 1 1"/>
-        </material>
-      </visual>
-    </link>
+    <link name="rear_light_link"/>
     <joint name="body_to_cover_joint" type="fixed">
       <origin xyz="0.0 0.0 0.1715" rpy="0.0 0.0 0.0" />
