Commit message: Apply some Dawid suggestions

File: panther_description/urdf/body.urdf.xacro (robot description, xacro)
@@ -42,5 +42,5 @@
     <link name="imu_link" />
     <joint name="body_to_front_bumper_joint" type="fixed">
-      <origin xyz="0.363 0.0 0.0" rpy="0.0 0.0 0.0" />
+      <origin xyz="0.362 0.0 0.0" rpy="0.0 0.0 0.0" />
       <parent link="body_link" />
       <child link="front_bumper_link" />
@@ -52,7 +52,7 @@
       <child link="front_light_link" />
     </joint>
-    <link name="front_light_link"/>
+    <link name="front_light_link" />
     <joint name="body_to_rear_bumper_joint" type="fixed">
-      <origin xyz="-0.363 0.0 0.0" rpy="0.0 0.0 ${pi}" />
+      <origin xyz="-0.362 0.0 0.0" rpy="0.0 0.0 ${pi}" />
       <parent link="body_link" />
       <child link="rear_bumper_link" />
@@ -64,5 +64,5 @@
       <child link="rear_light_link" />
     </joint>
-    <link name="rear_light_link"/>
+    <link name="rear_light_link" />
     <joint name="body_to_cover_joint" type="fixed">
       <origin xyz="0.0 0.0 0.1715" rpy="0.0 0.0 0.0" />

Commit message: Fix imu tf frame

File: panther_description/urdf/body.urdf.xacro (robot description, xacro)
@@ -4,7 +4,5 @@
   <xacro:macro
     name="body"
-    params="wheel_radius
-            imu_pos_x imu_pos_y imu_pos_z
-            imu_rot_r imu_rot_p imu_rot_y">
+    params="wheel_radius imu_xyz imu_rpy">
     <link name="base_link" />
     <joint name="base_to_body_joint" type="fixed">
@@ -35,6 +33,5 @@
     </link>
     <joint name="body_to_imu_joint" type="fixed">
-      <origin xyz="${imu_pos_x} ${imu_pos_y} ${imu_pos_z}"
-        rpy="${imu_rot_r} ${imu_rot_p} ${imu_rot_y}" />
+      <origin xyz="${imu_xyz}" rpy="${imu_rpy}" />
       <parent link="body_link" />
       <child link="imu_link" />

File: panther_description/urdf/gazebo.urdf.xacro (robot description, xacro)
@@ -5,10 +5,5 @@
     <!-- Read property -->
     <xacro:property name="battery_config" value="${xacro.load_yaml(config_file)}" />
-    <xacro:if value="${namespace == ''}">
-      <xacro:property name="ns" value="" />
-    </xacro:if>
-    <xacro:unless value="${namespace == ''}">
-        <xacro:property name="ns" value="${namespace}/" />
-    </xacro:unless>
+    <xacro:property name="ns" value='${namespace + "/" if namespace else ""}' />
     <!-- Sim Battery -->
     <gazebo>
@@ -59,10 +54,5 @@
   <!-- IMU specification: https://www.phidgets.com/?tier=3&catid=10&pcid=8&prodid=1025#Tab_Specifications -->
   <xacro:macro name="imu" params="reference_frame namespace:=''">
-    <xacro:if value="${namespace == ''}">
-      <xacro:property name="ns" value="" />
-    </xacro:if>
-    <xacro:unless value="${namespace == ''}">
-        <xacro:property name="ns" value="${namespace}/" />
-    </xacro:unless>
+    <xacro:property name="ns" value='${namespace + "/" if namespace else ""}' />
     <gazebo reference="${reference_frame}">
       <sensor name="${ns}imu" type="imu">

File: panther_description/urdf/panther.urdf.xacro (robot description, xacro)
@@ -5,10 +5,4 @@
   <!-- if lidars have to work correctly, use_gpu has to be true. -->
   <xacro:arg name="use_gpu" default="true" />
-  <xacro:arg name="imu_pos_x" default="0.169" />
-  <xacro:arg name="imu_pos_y" default="0.025" />
-  <xacro:arg name="imu_pos_z" default="0.092" />
-  <xacro:arg name="imu_rot_r" default="0.0" />
-  <xacro:arg name="imu_rot_p" default="0.0" />
-  <xacro:arg name="imu_rot_y" default="-1.57" />
   <xacro:arg name="wheel_config_file"
     default="$(find panther_description)/config/WH01.yaml" />
@@ -22,10 +16,4 @@
     panther_version="$(arg panther_version)"
     use_sim="$(arg use_sim)"
-    imu_pos_x="$(arg imu_pos_x)"
-    imu_pos_y="$(arg imu_pos_y)"
-    imu_pos_z="$(arg imu_pos_z)"
-    imu_rot_r="$(arg imu_rot_r)"
-    imu_rot_p="$(arg imu_rot_p)"
-    imu_rot_y="$(arg imu_rot_y)"
     wheel_config_file="$(arg wheel_config_file)"
     controller_config_file="$(arg controller_config_file)"

File: panther_description/urdf/panther_macro.urdf.xacro (robot description, xacro)
@@ -8,17 +8,14 @@
             battery_config_file
             use_sim:=false
-            imu_pos_x:=0.168
-            imu_pos_y:=0.028
-            imu_pos_z:=0.083
-            imu_rot_r:=3.14
-            imu_rot_p:=-1.57
-            imu_rot_y:=0.0
             namespace:=''">
-    <xacro:if value="${namespace == ''}">
-      <xacro:property name="ns" value="" />
+    <xacro:if value="${float(panther_version) >= 1.0}" >
+      <xacro:property name="imu_xyz" value="0.168 0.028 0.083" lazy_eval="false"/>
+      <xacro:property name="imu_rpy" value="3.14 -1.57 0.0" lazy_eval="false"/>
     </xacro:if>
-    <xacro:unless value="${namespace == ''}">
-        <xacro:property name="ns" value="${namespace}/" />
-    </xacro:unless>
+    <xacro:if value="${float(panther_version) > 1.06}">
+      <xacro:property name="imu_xyz" value="-0.195 0.010 0.085" />
+      <xacro:property name="imu_rpy" value="0.000 -0.000 3.142" />
+    </xacro:if>
+    <xacro:property name="ns" value='${namespace + "/" if namespace else ""}' />
     <xacro:property name="wheel_config" value="${xacro.load_yaml(wheel_config_file)}" />
     <xacro:property name="wheel_separation_x" value="0.44" />
@@ -30,10 +27,6 @@
     <xacro:body.body
       wheel_radius="${wheel_config['wheel_radius']}"
-      imu_pos_x="${imu_pos_x}"
-      imu_pos_y="${imu_pos_y}"
-      imu_pos_z="${imu_pos_z}"
-      imu_rot_r="${imu_rot_r}"
-      imu_rot_p="${imu_rot_p}"
-      imu_rot_y="${imu_rot_y}" />
+      imu_xyz="${imu_xyz}"
+      imu_rpy="${imu_rpy}" />
     <!-- WHEEL DECLARATION -->
     <xacro:wheel.wheel

Commit message: changed lights links
Signed-off-by: Jakub Delicat <jakub.delicat@husarion.com>

File: panther_description/urdf/body.urdf.xacro (robot description, xacro)
@@ -47,10 +47,10 @@
     </joint>
     <link name="front_bumper_link" />
-    <joint name="front_bumper_to_front_light_joint" type="fixed">
+    <joint name="front_bumper_to_lights_channel_1_joint" type="fixed">
       <origin xyz="0.0 0.0 0.0185" rpy="0.0 0.0 0.0" />
       <parent link="front_bumper_link" />
-      <child link="front_light_link" />
+      <child link="lights_channel_1_link" />
     </joint>
-    <link name="front_light_link" />
+    <link name="lights_channel_1_link" />
     <joint name="body_to_rear_bumper_joint" type="fixed">
       <origin xyz="-0.362 0.0 0.0" rpy="0.0 0.0 ${pi}" />
@@ -59,10 +59,10 @@
     </joint>
     <link name="rear_bumper_link" />
-    <joint name="rear_bumper_to_rear_light_joint" type="fixed">
+    <joint name="rear_bumper_to_lights_channel_2_joint" type="fixed">
       <origin xyz="0.0 0.0 0.0185" rpy="0.0 0.0 0.0" />
       <parent link="rear_bumper_link" />
-      <child link="rear_light_link" />
+      <child link="lights_channel_2_link" />
     </joint>
-    <link name="rear_light_link" />
+    <link name="lights_channel_2_link" />
     <joint name="body_to_cover_joint" type="fixed">
       <origin xyz="0.0 0.0 0.1715" rpy="0.0 0.0 0.0" />

Commit message: Ros2 system status tf namespace (#372)
* Fix mecanum prefixes

Signed-off-by: Jakub Delicat <jakub.delicat@husarion.com>

* fixed frames

Signed-off-by: Jakub Delicat <jakub.delicat@husarion.com>

* Added mecanum argument | added y friction to normal wheels

Signed-off-by: Jakub Delicat <jakub.delicat@husarion.com>

* Added AddNamespaceToFrameID ros util and applied to system_status

Signed-off-by: Jakub Delicat <jakub.delicat@husarion.com>

* added tests

Signed-off-by: Jakub Delicat <jakub.delicat@husarion.com>

* Added prefix to images

Signed-off-by: Jakub Delicat <jakub.delicat@husarion.com>

* changed lights links

Signed-off-by: Jakub Delicat <jakub.delicat@husarion.com>

---------

Signed-off-by: Jakub Delicat <jakub.delicat@husarion.com>

File: panther_description/urdf/body.urdf.xacro (robot description, xacro)
@@ -44,10 +44,10 @@
     </joint>
     <link name="front_bumper_link" />
-    <joint name="front_bumper_to_front_light_joint" type="fixed">
+    <joint name="front_bumper_to_lights_channel_1_joint" type="fixed">
       <origin xyz="0.0 0.0 0.0185" rpy="0.0 0.0 0.0" />
       <parent link="front_bumper_link" />
-      <child link="front_light_link" />
+      <child link="lights_channel_1_link" />
     </joint>
-    <link name="front_light_link" />
+    <link name="lights_channel_1_link" />
     <joint name="body_to_rear_bumper_joint" type="fixed">
       <origin xyz="-0.362 0.0 0.0" rpy="0.0 0.0 ${pi}" />
@@ -56,10 +56,10 @@
     </joint>
     <link name="rear_bumper_link" />
-    <joint name="rear_bumper_to_rear_light_joint" type="fixed">
+    <joint name="rear_bumper_to_lights_channel_2_joint" type="fixed">
       <origin xyz="0.0 0.0 0.0185" rpy="0.0 0.0 0.0" />
       <parent link="rear_bumper_link" />
-      <child link="rear_light_link" />
+      <child link="lights_channel_2_link" />
     </joint>
-    <link name="rear_light_link" />
+    <link name="lights_channel_2_link" />
     <joint name="body_to_cover_joint" type="fixed">
       <origin xyz="0.0 0.0 0.1715" rpy="0.0 0.0 0.0" />

Commit message: Merge remote-tracking branch 'origin/ros2-devel' into ros2-testing-poc

File: panther_description/urdf/body.urdf.xacro (robot description, xacro)
@@ -4,7 +4,5 @@
   <xacro:macro
     name="body"
-    params="wheel_radius
-            imu_pos_x imu_pos_y imu_pos_z
-            imu_rot_r imu_rot_p imu_rot_y">
+    params="wheel_radius imu_xyz imu_rpy">
     <link name="base_link" />
     <joint name="base_to_body_joint" type="fixed">
@@ -35,6 +33,5 @@
     </link>
     <joint name="body_to_imu_joint" type="fixed">
-      <origin xyz="${imu_pos_x} ${imu_pos_y} ${imu_pos_z}"
-        rpy="${imu_rot_r} ${imu_rot_p} ${imu_rot_y}" />
+      <origin xyz="${imu_xyz}" rpy="${imu_rpy}" />
       <parent link="body_link" />
       <child link="imu_link" />
@@ -47,10 +44,10 @@
     </joint>
     <link name="front_bumper_link" />
-    <joint name="front_bumper_to_front_light_joint" type="fixed">
-      <origin xyz="0.0 0.0 0.0185" rpy="${pi/2} 0.0 ${pi/2}" />
+    <joint name="front_bumper_to_lights_channel_1_joint" type="fixed">
+      <origin xyz="0.0 0.0 0.0185" rpy="0.0 0.0 0.0" />
       <parent link="front_bumper_link" />
-      <child link="front_light_link" />
+      <child link="lights_channel_1_link" />
     </joint>
-    <link name="front_light_link" />
+    <link name="lights_channel_1_link" />
     <joint name="body_to_rear_bumper_joint" type="fixed">
       <origin xyz="-0.362 0.0 0.0" rpy="0.0 0.0 ${pi}" />
@@ -59,10 +56,10 @@
     </joint>
     <link name="rear_bumper_link" />
-    <joint name="rear_bumper_to_rear_light_joint" type="fixed">
-      <origin xyz="0.0 0.0 0.0185" rpy="${pi/2} 0.0 ${pi/2}" />
+    <joint name="rear_bumper_to_lights_channel_2_joint" type="fixed">
+      <origin xyz="0.0 0.0 0.0185" rpy="0.0 0.0 0.0" />
       <parent link="rear_bumper_link" />
-      <child link="rear_light_link" />
+      <child link="lights_channel_2_link" />
     </joint>
-    <link name="rear_light_link" />
+    <link name="lights_channel_2_link" />
     <joint name="body_to_cover_joint" type="fixed">
       <origin xyz="0.0 0.0 0.1715" rpy="0.0 0.0 0.0" />

File: panther_description/urdf/gazebo.urdf.xacro (robot description, xacro)
@@ -15,5 +15,5 @@
       <plugin filename="ignition-gazebo-linearbatteryplugin-system"
         name="gz::sim::systems::LinearBatteryPlugin">
-        <battery_name>${ns}panther_battery</battery_name>
+        <battery_name>${ns}battery</battery_name>
         <voltage>41.4</voltage>
         <open_circuit_voltage_constant_coef>42.0</open_circuit_voltage_constant_coef>
@@ -29,7 +29,4 @@
         <power_load>${battery_config['power_load']/100.0}</power_load>
         <start_draining>${battery_config['simulate_discharging']}</start_draining>
-        <ros>
-          <namespace>${namespace}</namespace>
-        </ros>
       </plugin>
     </gazebo>
@@ -43,6 +40,6 @@
           <namespace>${namespace}</namespace>
           <remapping>imu_broadcaster/imu:=imu/data</remapping>
-          <remapping>panther_base_controller/cmd_vel_unstamped:=cmd_vel</remapping>
-          <remapping>panther_base_controller/odom:=odom/wheels</remapping>
+          <remapping>drive_controller/cmd_vel_unstamped:=cmd_vel</remapping>
+          <remapping>drive_controller/odom:=odometry/wheels</remapping>
         </ros>
       </plugin>
@@ -75,7 +72,9 @@
         <visualize>false</visualize>
         <enable_metrics>false</enable_metrics>
-        <frame_id>imu_link</frame_id>
         <ignition_frame_id>imu_link</ignition_frame_id>
         <imu>
+          <orientation_reference_frame>
+            <localization>ENU</localization>
+          </orientation_reference_frame>
           <angular_velocity>
             <!-- rad/s -->
@@ -106,3 +105,21 @@
     </gazebo>
   </xacro:macro>
+  <!-- Lights -->
+  <xacro:macro name="light" params="reference_frame name namespace:=''">
+    <gazebo reference="${reference_frame}">
+      <light name="${name}" type="spot">
+        <cast_shadows>true</cast_shadows>
+        <visualize>0</visualize>
+        <diffuse>1.0 1.0 1.0</diffuse>
+        <specular>1.0 1.0 1.0</specular>
+        <direction>1 0 0</direction>
+        <intensity>1.0</intensity>
+        <spot>
+          <inner_angle>1.0</inner_angle>
+          <outer_angle>2.0</outer_angle>
+          <falloff>0.4</falloff>
+        </spot>
+      </light>
+    </gazebo>
+  </xacro:macro>
 </robot>

File: panther_description/urdf/panther_macro.urdf.xacro (robot description, xacro)
@@ -8,11 +8,11 @@
             battery_config_file
             use_sim:=false
-            imu_pos_x:=0.168
-            imu_pos_y:=0.028
-            imu_pos_z:=0.083
-            imu_rot_r:=3.14
-            imu_rot_p:=-1.57
-            imu_rot_y:=0.0
+            imu_xyz:='0.169 0.025 0.092'
+            imu_rpy:='0.0 0.0 -1.57'
             namespace:=''">
+    <xacro:if value="${use_sim}">
+      <xacro:property name="imu_xyz" value="-0.195 0.010 0.085" />
+      <xacro:property name="imu_rpy" value="0.000 -0.000 3.142" />
+    </xacro:if>
     <xacro:if value="${namespace == ''}">
       <xacro:property name="ns" value="" />
@@ -30,10 +30,6 @@
     <xacro:body.body
       wheel_radius="${wheel_config['wheel_radius']}"
-      imu_pos_x="${imu_pos_x}"
-      imu_pos_y="${imu_pos_y}"
-      imu_pos_z="${imu_pos_z}"
-      imu_rot_r="${imu_rot_r}"
-      imu_rot_p="${imu_rot_p}"
-      imu_rot_y="${imu_rot_y}" />
+      imu_xyz="${imu_xyz}"
+      imu_rpy="${imu_rpy}" />
     <!-- WHEEL DECLARATION -->
     <xacro:wheel.wheel
@@ -166,4 +162,6 @@
       <xacro:gazebo.controller config_file="${controller_config_file}" namespace="${namespace}" />
       <xacro:gazebo.imu reference_frame="imu_link" namespace="${namespace}" />
+      <xacro:gazebo.light reference_frame="lights_channel_1_link" name="lights_channel_1" namespace="${namespace}" />
+      <xacro:gazebo.light reference_frame="lights_channel_2_link" name="lights_channel_2" namespace="${namespace}" />
     </xacro:if>
   </xacro:macro>
