Commit message: Format

File: panther_description/urdf/gazebo.urdf.xacro (robot description, xacro)
@@ -16,5 +16,6 @@
     <!-- Sim Battery -->
     <gazebo>
-      <plugin filename="ignition-gazebo-linearbatteryplugin-system" name="gz::sim::systems::LinearBatteryPlugin">
+      <plugin filename="ignition-gazebo-linearbatteryplugin-system"
+        name="gz::sim::systems::LinearBatteryPlugin">
         <battery_name>panther_battery</battery_name>
         <voltage>41.4</voltage>
@@ -48,5 +49,6 @@
   </xacro:macro>
   <!-- IMU - noise -->
-  <xacro:macro name="gauss_noise" params="mean:=0.0 stddev:=0.0 bias_mean:=0.0 bias_stddev:=0.0 precision:=0.0">
+  <xacro:macro name="gauss_noise"
+    params="mean:=0.0 stddev:=0.0 bias_mean:=0.0 bias_stddev:=0.0 precision:=0.0">
     <noise type="gaussian">
       <mean>${mean}</mean>
@@ -73,22 +75,22 @@
           <angular_velocity>
             <x>
-              <xacro:gauss_noise stddev="0.01" bias_mean="3.3e-5" precision="1.2e-3"/>
+              <xacro:gauss_noise stddev="0.01" bias_mean="3.3e-5" precision="1.2e-3" />
             </x>
             <y>
-              <xacro:gauss_noise stddev="0.01" bias_mean="3.3e-5" precision="1.2e-3"/>
+              <xacro:gauss_noise stddev="0.01" bias_mean="3.3e-5" precision="1.2e-3" />
             </y>
             <z>
-              <xacro:gauss_noise stddev="0.01" bias_mean="3.3e-5" precision="1.2e-3"/>
+              <xacro:gauss_noise stddev="0.01" bias_mean="3.3e-5" precision="1.2e-3" />
             </z>
           </angular_velocity>
           <linear_acceleration>
             <x>
-              <xacro:gauss_noise stddev="2.8e-3" bias_mean="1.9e-3" precision="9.8e-4"/>
+              <xacro:gauss_noise stddev="2.8e-3" bias_mean="1.9e-3" precision="9.8e-4" />
             </x>
             <y>
-              <xacro:gauss_noise stddev="2.8e-3" bias_mean="1.9e-3" precision="9.8e-4"/>
+              <xacro:gauss_noise stddev="2.8e-3" bias_mean="1.9e-3" precision="9.8e-4" />
             </y>
             <z>
-              <xacro:gauss_noise stddev="2.8e-3" bias_mean="1.9e-3" precision="9.8e-4"/>
+              <xacro:gauss_noise stddev="2.8e-3" bias_mean="1.9e-3" precision="9.8e-4" />
             </z>
           </linear_acceleration>

File: panther_description/urdf/panther_macro.urdf.xacro (robot description, xacro)
@@ -109,7 +109,7 @@
     </ros2_control>
     <xacro:if value="${use_sim}">
-      <xacro:gazebo.battery config_file="${battery_config_file}"/>
-      <xacro:gazebo.controller config_file="${controller_config_file}"/>
-      <xacro:gazebo.imu reference_frame="imu_link" name="imu"/>
+      <xacro:gazebo.battery config_file="${battery_config_file}" />
+      <xacro:gazebo.controller config_file="${controller_config_file}" />
+      <xacro:gazebo.imu reference_frame="imu_link" name="imu" />
     </xacro:if>
   </xacro:macro>

Commit message: Preparation for namespace

File: panther_description/urdf/gazebo.urdf.xacro (robot description, xacro)
@@ -2,5 +2,5 @@
 <robot xmlns:xacro="http://wiki.ros.org/xacro">
   <!-- Battery -->
-  <xacro:macro name="battery" params="config_file">
+  <xacro:macro name="battery" params="config_file namespace:=''">
     <!-- Read property -->
     <xacro:property name="battery_config" value="${xacro.load_yaml(config_file)}" />
@@ -33,15 +33,19 @@
         <!-- https://github.com/gazebosim/gz-sim/issues/225 -->
         <fix_issue_225>true</fix_issue_225>
+        <ros>
+          <namespace>${namespace}</namespace>
+        </ros>
       </plugin>
     </gazebo>
   </xacro:macro>
   <!-- Controller -->
-  <xacro:macro name="controller" params="config_file">
+  <xacro:macro name="controller" params="config_file namespace:=''">
     <gazebo>
-      <plugin filename="ign_ros2_control-system"
-        name="ign_ros2_control::IgnitionROS2ControlPlugin">
+      <plugin filename="ign_ros2_control-system" name="ign_ros2_control::IgnitionROS2ControlPlugin">
         <parameters>${config_file}</parameters>
         <ros>
+          <namespace>${namespace}</namespace>
           <remapping>/panther_base_controller/cmd_vel_unstamped:=/cmd_vel</remapping>
+          <remapping>/tf:=tf</remapping>
         </ros>
       </plugin>
@@ -61,7 +65,13 @@
   <!-- IMU -->
   <!-- Noise ref: https://www.phidgets.com/?tier=3&catid=10&pcid=8&prodid=1025#Tab_Specifications -->
-  <xacro:macro name="imu" params="reference_frame name:='imu'">
+  <xacro:macro name="imu" params="reference_frame namespace:=''">
+    <xacro:if value="${namespace == ''}">
+      <xacro:property name="ns" value="" />
+    </xacro:if>
+    <xacro:unless value="${namespace == ''}">
+        <xacro:property name="ns" value="${namespace}/" />
+    </xacro:unless>
     <gazebo reference="${reference_frame}">
-      <sensor name="${name}" type="imu">
+      <sensor name="${ns}imu" type="imu">
         <plugin filename="ignition-gazebo-imu-system" name="ignition::gazebo::systems::Imu" />
         <always_on>true</always_on>
@@ -72,4 +82,7 @@
         <frame_id>imu_link</frame_id>
         <ignition_frame_id>imu_link</ignition_frame_id>
+        <ros>
+          <namespace>${namespace}</namespace>
+        </ros>
         <imu>
           <angular_velocity>

File: panther_description/urdf/panther.urdf.xacro (robot description, xacro)
@@ -17,4 +17,5 @@
   <xacro:arg name="battery_config_file"
     default="$(find panther_description)/config/battery_ign_plugin.yaml" />
+  <xacro:arg name="namespace" default="" />
   <xacro:include filename="$(find panther_description)/urdf/panther_macro.urdf.xacro" ns="husarion" />
   <xacro:husarion.panther_robot
@@ -30,4 +31,5 @@
     wheel_config_file="$(arg wheel_config_file)"
     controller_config_file="$(arg controller_config_file)"
-    battery_config_file="$(arg battery_config_file)" />
+    battery_config_file="$(arg battery_config_file)"
+    namespace="$(arg namespace)" />
 </robot>

File: panther_description/urdf/panther_macro.urdf.xacro (robot description, xacro)
@@ -14,5 +14,12 @@
             imu_rot_p:=-1.57
             imu_rot_y:=0.0
-            simulation_engine:='ignition-gazebo'">
+            simulation_engine:='ignition-gazebo'
+            namespace:=''">
+    <xacro:if value="${namespace == ''}">
+      <xacro:property name="ns" value="" />
+    </xacro:if>
+    <xacro:unless value="${namespace == ''}">
+        <xacro:property name="ns" value="${namespace}/" />
+    </xacro:unless>
     <xacro:property name="wheel_config" value="${xacro.load_yaml(wheel_config_file)}" />
     <xacro:property name="wheel_separation_x" value="0.44" />
@@ -47,5 +54,5 @@
       wheel_separation_x="${wheel_separation_x}"
       prefix="rr" />
-    <ros2_control name="wheels" type="system">
+    <ros2_control name="${ns}wheels" type="system">
       <hardware>
         <xacro:if value="${use_sim}">
@@ -109,5 +116,5 @@
       </joint>
       <xacro:if value="${use_sim}">
-        <sensor name="imu">
+        <sensor name="${ns}imu">
           <state_interface name="orientation.x" />
           <state_interface name="orientation.y" />
@@ -124,7 +131,7 @@
     </ros2_control>
     <xacro:if value="${use_sim}">
-      <xacro:gazebo.battery config_file="${battery_config_file}" />
-      <xacro:gazebo.controller config_file="${controller_config_file}" />
-      <xacro:gazebo.imu reference_frame="imu_link" name="imu" />
+      <xacro:gazebo.battery config_file="${battery_config_file}" namespace="${namespace}" />
+      <xacro:gazebo.controller config_file="${controller_config_file}" namespace="${namespace}" />
+      <xacro:gazebo.imu reference_frame="imu_link" namespace="${namespace}" />
     </xacro:if>
   </xacro:macro>

Commit message: Ros2 namespace (#255)
* Preparation for namespace

* Simulation working

* Hardware look ok

* Update panther_controller/config/WH01_controller.yaml

Co-authored-by: Jakub Delicat <109142865+delihus@users.noreply.github.com>

* Apply Jakub suggestions

Co-authored-by: Jakub Delicat <109142865+delihus@users.noreply.github.com>

* Fix imu

* Readme

* Add imu namespace

* Jakub suggestions

* Add panther manager to xml

* pre-commit

* Fixed ekf

Signed-off-by: Jakub Delicat <jakub.delicat@husarion.com>

* Additional remapping

* fix imu

* Pawel suggestions (collision with gamepad)

* cmd_vel

* Use namespace instead of PushRosNamespace

---------

Signed-off-by: Jakub Delicat <jakub.delicat@husarion.com>
Co-authored-by: Jakub Delicat <109142865+delihus@users.noreply.github.com>
Co-authored-by: Jakub Delicat <jakub.delicat@husarion.com>

File: panther_description/urdf/gazebo.urdf.xacro (robot description, xacro)
@@ -2,5 +2,5 @@
 <robot xmlns:xacro="http://wiki.ros.org/xacro">
   <!-- Battery -->
-  <xacro:macro name="battery" params="config_file">
+  <xacro:macro name="battery" params="config_file namespace:=''">
     <!-- Read property -->
     <xacro:property name="battery_config" value="${xacro.load_yaml(config_file)}" />
@@ -33,17 +33,20 @@
         <!-- https://github.com/gazebosim/gz-sim/issues/225 -->
         <fix_issue_225>true</fix_issue_225>
+        <ros>
+          <namespace>${namespace}</namespace>
+        </ros>
       </plugin>
     </gazebo>
   </xacro:macro>
   <!-- Controller -->
-  <xacro:macro name="controller" params="config_file">
+  <xacro:macro name="controller" params="config_file namespace:=''">
     <gazebo>
-      <plugin filename="ign_ros2_control-system"
-        name="ign_ros2_control::IgnitionROS2ControlPlugin">
+      <plugin filename="ign_ros2_control-system" name="ign_ros2_control::IgnitionROS2ControlPlugin">
         <parameters>${config_file}</parameters>
         <ros>
-          <remapping>panther_base_controller/cmd_vel_unstamped:=/cmd_vel</remapping>
+          <namespace>${namespace}</namespace>
+          <remapping>imu_broadcaster/imu:=imu/data</remapping>
+          <remapping>panther_base_controller/cmd_vel_unstamped:=cmd_vel</remapping>
           <remapping>panther_base_controller/odom:=odom/wheels</remapping>
-          <remapping>/imu_broadcaster/imu:=imu/data</remapping>
         </ros>
       </plugin>
@@ -62,11 +65,17 @@
   </xacro:macro>
   <!-- IMU specification: https://www.phidgets.com/?tier=3&catid=10&pcid=8&prodid=1025#Tab_Specifications -->
-  <xacro:macro name="imu" params="reference_frame name:='imu'">
+  <xacro:macro name="imu" params="reference_frame namespace:=''">
+    <xacro:if value="${namespace == ''}">
+      <xacro:property name="ns" value="" />
+    </xacro:if>
+    <xacro:unless value="${namespace == ''}">
+        <xacro:property name="ns" value="${namespace}/" />
+    </xacro:unless>
     <gazebo reference="${reference_frame}">
-      <sensor name="${name}" type="imu">
+      <sensor name="${ns}imu" type="imu">
         <plugin filename="ignition-gazebo-imu-system" name="ignition::gazebo::systems::Imu" />
         <always_on>true</always_on>
         <update_rate>50</update_rate>
-        <topic>imu/data_raw</topic>
+        <topic>${ns}imu/data_raw</topic>
         <visualize>false</visualize>
         <enable_metrics>false</enable_metrics>

Commit message: Added components
Signed-off-by: Jakub Delicat <jakub.delicat@husarion.com>

File: panther_description/urdf/gazebo.urdf.xacro (robot description, xacro)
@@ -74,5 +74,4 @@
     <gazebo reference="${reference_frame}">
       <sensor name="${ns}imu" type="imu">
-        <plugin filename="ignition-gazebo-imu-system" name="ignition::gazebo::systems::Imu" />
         <always_on>true</always_on>
         <update_rate>50</update_rate>

File: panther_description/urdf/panther.urdf.xacro (robot description, xacro)
@@ -3,5 +3,6 @@
   <xacro:arg name="panther_version" default="1.0" />
   <xacro:arg name="use_sim" default="false" />
-  <xacro:arg name="use_gpu" default="false" />
+  <!-- if lidars have to work correctly, use_gpu has to be true. -->
+  <xacro:arg name="use_gpu" default="true" />
   <xacro:arg name="imu_pos_x" default="0.169" />
   <xacro:arg name="imu_pos_y" default="0.025" />
@@ -33,3 +34,15 @@
     battery_config_file="$(arg battery_config_file)"
     namespace="$(arg namespace)" />
+  <xacro:arg name="components_config_path" default="$(find panther_bringup)/config/components.yaml" />
+  <xacro:property name="components_config_path_property" value="$(arg components_config_path)" />
+  <xacro:unless value="${components_config_path_property == 'None'}">
+    <xacro:include filename="$(find ros_components_description)/urdf/components.urdf.xacro"
+      ns="husarion_components" />
+    <xacro:husarion_components.create_components
+      components_config_path="${components_config_path_property}"
+      use_gpu="$(arg use_gpu)"
+      simulation_engine="$(arg simulation_engine)"
+      namespace="$(arg namespace)"
+    />
+  </xacro:unless>
 </robot>

Commit message: Fix battery discharge

File: panther_description/urdf/gazebo.urdf.xacro (robot description, xacro)
@@ -5,12 +5,9 @@
     <!-- Read property -->
     <xacro:property name="battery_config" value="${xacro.load_yaml(config_file)}" />
-    <xacro:property name="bat_initial_charge"
-      value="${20.0*battery_config['initial_charge_percentage']/100.0}" />
-    <xacro:property name="bat_charging_time" value="${battery_config['charging_time']}" />
-    <xacro:if value="${battery_config['simulate_discharging']}">
-      <xacro:property name="bat_power_load" value="${battery_config['power_load']}" />
+    <xacro:if value="${namespace == ''}">
+      <xacro:property name="ns" value="" />
     </xacro:if>
-    <xacro:unless value="${battery_config['simulate_discharging']}">
-      <xacro:property name="bat_power_load" value="0.0" />
+    <xacro:unless value="${namespace == ''}">
+        <xacro:property name="ns" value="${namespace}/" />
     </xacro:unless>
     <!-- Sim Battery -->
@@ -18,19 +15,18 @@
       <plugin filename="ignition-gazebo-linearbatteryplugin-system"
         name="gz::sim::systems::LinearBatteryPlugin">
-        <battery_name>panther_battery</battery_name>
+        <battery_name>${ns}panther_battery</battery_name>
         <voltage>41.4</voltage>
         <open_circuit_voltage_constant_coef>42.0</open_circuit_voltage_constant_coef>
         <open_circuit_voltage_linear_coef>-10.0</open_circuit_voltage_linear_coef>
-        <initial_charge>${bat_initial_charge}</initial_charge>
-        <capacity>20.0</capacity>
+        <initial_charge>${battery_config['initial_charge_percentage']*battery_config['capacity']}</initial_charge>
+        <capacity>${battery_config['capacity']}</capacity>
         <resistance>0.15</resistance>
         <smooth_current_tau>2.0</smooth_current_tau>
         <enable_recharge>true</enable_recharge>
-        <charging_time>${bat_charging_time}</charging_time>
+        <charging_time>${battery_config['charging_time']}</charging_time>
         <soc_threshold>2.0</soc_threshold>
-        <power_load>${bat_power_load}</power_load>
-        <start_on_motion>false</start_on_motion>
-        <!-- https://github.com/gazebosim/gz-sim/issues/225 -->
-        <fix_issue_225>true</fix_issue_225>
+        <!-- Because of https://github.com/gazebosim/gz-sim/issues/225 devision by 100-->
+        <power_load>${battery_config['power_load']/100.0}</power_load>
+        <start_draining>${battery_config['simulate_discharging']}</start_draining>
         <ros>
           <namespace>${namespace}</namespace>

Commit message: Ros2 add components (#277)
* Added components

Signed-off-by: Jakub Delicat <jakub.delicat@husarion.com>

* default config

Signed-off-by: Jakub Delicat <jakub.delicat@husarion.com>

* Delete unnecessary declaration

* added enter

Signed-off-by: Jakub Delicat <jakub.delicat@husarion.com>

* renamed gz_components

Signed-off-by: Jakub Delicat <jakub.delicat@husarion.com>

* removed simulation engine and use_gpu from components

Signed-off-by: Jakub Delicat <jakub.delicat@husarion.com>

* suggesion applied

Signed-off-by: Jakub Delicat <jakub.delicat@husarion.com>

* updated readme

Signed-off-by: Jakub Delicat <jakub.delicat@husarion.com>

---------

Signed-off-by: Jakub Delicat <jakub.delicat@husarion.com>
Co-authored-by: rafal-gorecki <rafal.gorecki@husarion.com>

File: panther_description/urdf/gazebo.urdf.xacro (robot description, xacro)
@@ -70,5 +70,4 @@
     <gazebo reference="${reference_frame}">
       <sensor name="${ns}imu" type="imu">
-        <plugin filename="ignition-gazebo-imu-system" name="ignition::gazebo::systems::Imu" />
         <always_on>true</always_on>
         <update_rate>50</update_rate>

File: panther_description/urdf/panther.urdf.xacro (robot description, xacro)
@@ -3,5 +3,6 @@
   <xacro:arg name="panther_version" default="1.0" />
   <xacro:arg name="use_sim" default="false" />
-  <xacro:arg name="use_gpu" default="false" />
+  <!-- if lidars have to work correctly, use_gpu has to be true. -->
+  <xacro:arg name="use_gpu" default="true" />
   <xacro:arg name="imu_pos_x" default="0.169" />
   <xacro:arg name="imu_pos_y" default="0.025" />
@@ -33,3 +34,13 @@
     battery_config_file="$(arg battery_config_file)"
     namespace="$(arg namespace)" />
+  <xacro:arg name="components_config_path" default="$(find panther_bringup)/config/components.yaml" />
+  <xacro:property name="components_config_path_property" value="$(arg components_config_path)" />
+  <xacro:unless value="${components_config_path_property == 'None'}">
+    <xacro:include filename="$(find ros_components_description)/urdf/components.urdf.xacro"
+      ns="husarion_components" />
+    <xacro:husarion_components.create_components
+      components_config_path="${components_config_path_property}"
+      namespace="$(arg namespace)"
+    />
+  </xacro:unless>
 </robot>

Commit message: Undo namespace

File: panther_description/urdf/gazebo.urdf.xacro (robot description, xacro)
@@ -5,5 +5,10 @@
     <!-- Read property -->
     <xacro:property name="battery_config" value="${xacro.load_yaml(config_file)}" />
-    <xacro:property name="ns" value='${namespace + "/" if namespace else ""}' />
+    <xacro:if value="${namespace == ''}">
+      <xacro:property name="ns" value="" />
+    </xacro:if>
+    <xacro:unless value="${namespace == ''}">
+        <xacro:property name="ns" value="${namespace}/" />
+    </xacro:unless>
     <!-- Sim Battery -->
     <gazebo>
@@ -54,5 +59,10 @@
   <!-- IMU specification: https://www.phidgets.com/?tier=3&catid=10&pcid=8&prodid=1025#Tab_Specifications -->
   <xacro:macro name="imu" params="reference_frame namespace:=''">
-    <xacro:property name="ns" value='${namespace + "/" if namespace else ""}' />
+    <xacro:if value="${namespace == ''}">
+      <xacro:property name="ns" value="" />
+    </xacro:if>
+    <xacro:unless value="${namespace == ''}">
+        <xacro:property name="ns" value="${namespace}/" />
+    </xacro:unless>
     <gazebo reference="${reference_frame}">
       <sensor name="${ns}imu" type="imu">

File: panther_description/urdf/panther_macro.urdf.xacro (robot description, xacro)
@@ -15,5 +15,10 @@
       <xacro:property name="imu_rpy" value="0.000 -0.000 3.142" />
     </xacro:if>
-    <xacro:property name="ns" value='${namespace + "/" if namespace else ""}' />
+    <xacro:if value="${namespace == ''}">
+      <xacro:property name="ns" value="" />
+    </xacro:if>
+    <xacro:unless value="${namespace == ''}">
+        <xacro:property name="ns" value="${namespace}/" />
+    </xacro:unless>
     <xacro:property name="wheel_config" value="${xacro.load_yaml(wheel_config_file)}" />
     <xacro:property name="wheel_separation_x" value="0.44" />

Commit message: Save work

File: panther_description/urdf/gazebo.urdf.xacro (robot description, xacro)
@@ -109,5 +109,15 @@
   </xacro:macro>
   <!-- Lights -->
-  <xacro:macro name="light" params="reference_frame name namespace:=''">
+  <xacro:macro name="light" params="reference_frame name topic namespace:=''">
+    <gazebo>
+      <plugin filename="LEDStrip" name="LEDStrip">
+        <light_name>${name}</light_name>
+        <topic>${topic}</topic>
+        <namespace>panther</namespace>
+        <frequency>10</frequency>
+        <width>0.5</width>
+        <height>0.015</height>
+      </plugin>
+    </gazebo>
     <gazebo reference="${reference_frame}">
       <light name="${name}" type="spot">

File: panther_description/urdf/panther_macro.urdf.xacro (robot description, xacro)
@@ -163,6 +163,6 @@
       <xacro:gazebo.controller config_file="${controller_config_file}" namespace="${namespace}" />
       <xacro:gazebo.imu reference_frame="imu_link" namespace="${namespace}" />
-      <xacro:gazebo.light reference_frame="lights_channel_1_link" name="lights_channel_1" namespace="${namespace}" />
-      <xacro:gazebo.light reference_frame="lights_channel_2_link" name="lights_channel_2" namespace="${namespace}" />
+      <xacro:gazebo.light reference_frame="lights_channel_1_link" name="lights_channel_1" topic="lights/channel_1_frame" namespace="${namespace}" />
+      <xacro:gazebo.light reference_frame="lights_channel_2_link" name="lights_channel_2" topic="lights/channel_2_frame" namespace="${namespace}" />
     </xacro:if>
   </xacro:macro>
