Commit message: review

File: lynx_description/urdf/wheel.urdf.xacro (robot description, xacro)
@@ -33,5 +33,5 @@
       <axis xyz="0.0 1.0 0.0" />
       <limit effort="64.5" velocity="10.958" />
-      <dynamics damping="0.01" friction="0.9" />
+      <dynamics damping="0.01" friction="0.1" />
     </joint>
     <link name="${prefix}_wheel_link">
@@ -64,4 +64,21 @@
       </inertial>
     </link>
+    <xacro:if value="${use_sim}">
+      <xacro:if value="${wheel_config['mecanum']}">
+        <gazebo reference="${prefix}_wheel_link" xmlns:ignition="http://ignitionrobotics.org/schema">
+          <collision>
+            <surface>
+              <friction>
+                <ode>
+                  <mu>1.0</mu>
+                  <mu2>0.0</mu2>
+                  <fdir1 ignition:expressed_in="base_link">${fdir}</fdir1>
+                </ode>
+              </friction>
+            </surface>
+          </collision>
+        </gazebo>
+      </xacro:if>
+    </xacro:if>
   </xacro:macro>
 </robot>
